File: hw/rev-a/kicad/CASS.kicad_sch (KiCad schematic)
At the start: 19 parts, among them J13 CASS_B_HEADER, J20 CASS_A_HEADER, J3 CASS A, J6 CASS B, Q2 AO3401A, Q3 AO3401A

Commit message: hw: correct Mouser PN for headers
Parts:
- J13, J20: MOUSER 649-1012937893602BLF -> 649-1012937891002BLF
Changed lines of the file:
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@@
       (effects (font (size 1.27 1.27)) hide)
     )
-    (property "MOUSER" "649-1012937893602BLF" (id 4) (at 195.58 44.45 0)
+    (property "MOUSER" "649-1012937891002BLF" (id 4) (at 195.58 44.45 0)
       (effects (font (size 1.27 1.27)) hide)
     )
@@
       (effects (font (size 1.27 1.27)) hide)
     )
-    (property "MOUSER" "649-1012937893602BLF" (id 4) (at 241.3 44.45 0)
-      (effects (font (size 1.27 1.27)) hide)
-    )
+    (property "MOUSER" "649-1012937891002BLF" (id 4) (at 241.3 44.45 0)
+      (effects (font (size 1.27 1.27)) hide)
+    )
