File: hw/rev-a/kicad/MCU.kicad_sch (KiCad schematic)
At the start: 34 parts, among them J25 MENU, SW4 RUN, SW5 MENU, U21 RP2040, Y1 12 MHz

Commit message: hw: correct Mouser PN for headers
Parts:
- J25: MOUSER 649-1012937893602BLF -> 649-1012937891002BLF
Changed lines of the file:
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@@
       (effects (font (size 1.27 1.27)) hide)
     )
-    (property "MOUSER" "649-1012937893602BLF" (id 4) (at 25.4 168.91 0)
+    (property "MOUSER" "649-1012937891002BLF" (id 4) (at 25.4 168.91 0)
       (effects (font (size 1.27 1.27)) hide)
     )
