File: hw/rev-a/kicad/POWER.kicad_sch (KiCad schematic)
At the start: 58 parts, among them J10 5V PWR, J11 9V POWER, J12 9V POWER, J8 PET POWER, U3 AMS1117-3.3, U4 XL1509-5.0E1, U5 LM317AG-TN3-R, U6 LM317AG-TN3-R

Commit message: hw: correct Mouser PN for headers
Parts:
- J11: MOUSER 649-1012937893602BLF -> 649-1012937891002BLF
Changed lines of the file:
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@@
       (effects (font (size 1.27 1.27)) hide)
     )
-    (property "MOUSER" "649-1012937893602BLF" (id 4) (at 95.25 41.91 0)
+    (property "MOUSER" "649-1012937891002BLF" (id 4) (at 95.25 41.91 0)
       (effects (font (size 1.27 1.27)) hide)
     )
