File: hw/rev-a/kicad/CPU.kicad_sch (KiCad schematic)
At the start: 12 parts, among them SW1 RESET, SW2 NMI, U1 W65C02S, U2 AS6C1008

Commit message: hw: DNP C23-C24
Parts:
- C23, C24: value 10u -> DNP; now left out of the parts list
Changed lines of the file:
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@@
   )
   (symbol (lib_id "Device:C_Small") (at 107.95 184.15 0) (unit 1)
-    (in_bom yes) (on_board yes)
+    (in_bom no) (on_board yes)
     (property "Reference" "C23" (id 0) (at 110.2868 182.9816 0)
       (effects (font (size 1.27 1.27)) (justify left))
     )
-    (property "Value" "10u" (id 1) (at 110.2868 185.293 0)
+    (property "Value" "DNP" (id 1) (at 110.2868 185.293 0)
       (effects (font (size 1.27 1.27)) (justify left))
     )
@@
   )
   (symbol (lib_id "Device:C_Small") (at 138.43 184.15 0) (unit 1)
-    (in_bom yes) (on_board yes)
+    (in_bom no) (on_board yes)
     (property "Reference" "C24" (id 0) (at 140.7668 182.9816 0)
       (effects (font (size 1.27 1.27)) (justify left))
     )
-    (property "Value" "10u" (id 1) (at 140.7668 185.293 0)
+    (property "Value" "DNP" (id 1) (at 140.7668 185.293 0)
       (effects (font (size 1.27 1.27)) (justify left))
     )
