File: hw/rev-c/mainboard/kicad/CASS.kicad_sch (KiCad schematic)
At the start: 19 parts, among them J13 CASS_B_HEADER, J20 CASS_A_HEADER, J3 CASS A, J6 CASS B, Q2 AO3401A, Q3 AO3401A

Commit message: hw: fix wire/grid violations in schematic
Parts:
- J3, J6: symbol Retrocomputing:CBM_PET_CASS_Conn_01x06_Card_Edge -> EconoPET:CBM_PET_CASS_Conn_01x06_Card_Edge
Changed lines of the file:
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@@
 	)
 	(symbol
-		(lib_id "Retrocomputing:CBM_PET_CASS_Conn_01x06_Card_Edge")
+		(lib_id "EconoPET:CBM_PET_CASS_Conn_01x06_Card_Edge")
 		(at 242.57 142.24 0)
 		(unit 1)
@@
 	)
 	(symbol
-		(lib_name "CBM_PET_CASS_Conn_01x06_Card_Edge_1")
-		(lib_id "Retrocomputing:CBM_PET_CASS_Conn_01x06_Card_Edge")
+		(lib_id "EconoPET:CBM_PET_CASS_Conn_01x06_Card_Edge")
 		(at 242.57 100.33 0)
 		(unit 1)

Commit message: hw: update diode and connector symbols
Parts:
- J13, J20: symbol Connector:Conn_01x06_Male -> Connector:Conn_01x06_Pin
Changed lines of the file:
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@@
 	)
 	(symbol
-		(lib_id "Connector:Conn_01x06_Male")
+		(lib_id "Connector:Conn_01x06_Pin")
 		(at 195.58 44.45 0)
 		(mirror y)
@@
 			)
 		)
-		(property "Description" ""
+		(property "Description" "Generic connector, single row, 01x06, script generated"
 			(at 195.58 44.45 0)
 			(effects
@@
 	)
 	(symbol
-		(lib_id "Connector:Conn_01x06_Male")
+		(lib_id "Connector:Conn_01x06_Pin")
 		(at 241.3 44.45 0)
 		(mirror y)
@@
 			)
 		)
-		(property "Description" ""
+		(property "Description" "Generic connector, single row, 01x06, script generated"
 			(at 241.3 44.45 0)
 			(effects

Commit message: hw: update more footprints
Parts:
- Q2, Q3: footprint JLCPCB:SOT-23_L2.9-W1.3-P1.90-LS2.4-BR -> EconoPET:SOT-23_L2.9-W1.3-P1.90-LS2.4-BR
Changed lines of the file:
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@@
 			)
 		)
-		(property "Footprint" "JLCPCB:SOT-23_L2.9-W1.3-P1.90-LS2.4-BR"
+		(property "Footprint" "EconoPET:SOT-23_L2.9-W1.3-P1.90-LS2.4-BR"
 			(at 211.455 90.17 0)
 			(effects
@@
 			)
 		)
-		(property "Footprint" "JLCPCB:SOT-23_L2.9-W1.3-P1.90-LS2.4-BR"
+		(property "Footprint" "EconoPET:SOT-23_L2.9-W1.3-P1.90-LS2.4-BR"
 			(at 211.455 132.08 0)
 			(effects

Commit message: hw: renumber reference designators
Parts:
- renumbered C75 to C76, J20 to J14, J13 to J15, J3 to J16, J6 to J17, R25 to R30, R26 to R31, R27 to R32, R28 to R33
Changed lines of the file:
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@@
 		(on_board yes)
 		(dnp no)
-		(property "Reference" "J6"
+		(property "Reference" "J17"
 			(at 247.142 142.4432 0)
 			(effects
@@
 			(project ""
 				(path "/2eea20e6-112c-411a-b615-885ae773135a/00000000-0000-0000-0000-000061bef9ce"
-					(reference "J6")
+					(reference "J17")
 					(unit 1)
 				)
@@
 		(on_board yes)
 		(dnp no)
-		(property "Reference" "J3"
+		(property "Reference" "J16"
 			(at 247.142 100.5332 0)
 			(effects
@@
 			(project ""
 				(path "/2eea20e6-112c-411a-b615-885ae773135a/00000000-0000-0000-0000-000061bef9ce"
-					(reference "J3")
+					(reference "J16")
 					(unit 1)
 				)
@@
 		(on_board yes)
 		(dnp no)
-		(property "Reference" "R25"
+		(property "Reference" "R30"
 			(at 51.435 106.045 90)
 			(effects
@@
 			(project ""
 				(path "/2eea20e6-112c-411a-b615-885ae773135a/00000000-0000-0000-0000-000061bef9ce"
-					(reference "R25")
+					(reference "R30")
 					(unit 1)
 				)
@@
 		(dnp no)
 		(fields_autoplaced yes)
-		(property "Reference" "J20"
+		(property "Reference" "J14"
 			(at 196.85 44.4499 0)
 			(effects
@@
 			(project ""
 				(path "/2eea20e6-112c-411a-b615-885ae773135a/00000000-0000-0000-0000-000061bef9ce"
-					(reference "J20")
+					(reference "J14")
 					(unit 1)
 				)
@@
 		(on_board yes)
 		(dnp no)
-		(property "Reference" "R27"
+		(property "Reference" "R32"
 			(at 197.0786 95.3516 0)
 			(effects
@@
 			(project ""
 				(path "/2eea20e6-112c-411a-b615-885ae773135a/00000000-0000-0000-0000-000061bef9ce"
-					(reference "R27")
+					(reference "R32")
 					(unit 1)
 				)
@@
 		(on_board yes)
 		(dnp no)
-		(property "Reference" "C75"
+		(property "Reference" "C76"
 			(at 36.6268 176.4284 0)
 			(effects
@@
 			(project ""
 				(path "/2eea20e6-112c-411a-b615-885ae773135a/00000000-0000-0000-0000-000061bef9ce"
-					(reference "C75")
+					(reference "C76")
 					(unit 1)
 				)
@@
 		(dnp no)
 		(fields_autoplaced yes)
-		(property "Reference" "J13"
+		(property "Reference" "J15"
 			(at 242.57 44.4499 0)
 			(effects
@@
 			(project ""
 				(path "/2eea20e6-112c-411a-b615-885ae773135a/00000000-0000-0000-0000-000061bef9ce"
-					(reference "J13")
+					(reference "J15")
 					(unit 1)
 				)
@@
 		(on_board yes)
 		(dnp no)
-		(property "Reference" "R28"
+		(property "Reference" "R33"
 			(at 197.0786 137.2616 0)
 			(effects
@@
 			(project ""
 				(path "/2eea20e6-112c-411a-b615-885ae773135a/00000000-0000-0000-0000-000061bef9ce"
-					(reference "R28")
+					(reference "R33")
 					(unit 1)
 				)
@@
 		(on_board yes)
 		(dnp no)
-		(property "Reference" "R26"
+		(property "Reference" "R31"
 			(at 51.435 111.125 90)
 			(effects
@@
 			(project ""
 				(path "/2eea20e6-112c-411a-b615-885ae773135a/00000000-0000-0000-0000-000061bef9ce"
-					(reference "R26")
-					(unit 1)
-				)
+					(reference "R31")
+					(unit 1)
+				)

Commit message: hw: match original PET designators for connectors
Parts:
- renumbered C76 to C77, J14 to J15, J15 to J16, J16 to J3, J17 to J6, JP2 to JP1, JP3 to JP2, JP4 to JP3, JP5 to JP4, JP6 to JP5, JP7 to JP6, R30 to R32, R31 to R33, R32 to R34, R33 to R35
Changed lines of the file:
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@@
 		(on_board yes)
 		(dnp no)
-		(property "Reference" "J17"
+		(property "Reference" "J6"
 			(at 247.142 142.4432 0)
 			(effects
@@
 			(project ""
 				(path "/2eea20e6-112c-411a-b615-885ae773135a/00000000-0000-0000-0000-000061bef9ce"
-					(reference "J17")
+					(reference "J6")
 					(unit 1)
 				)
@@
 		(on_board yes)
 		(dnp no)
-		(property "Reference" "J16"
+		(property "Reference" "J3"
 			(at 247.142 100.5332 0)
 			(effects
@@
 			(project ""
 				(path "/2eea20e6-112c-411a-b615-885ae773135a/00000000-0000-0000-0000-000061bef9ce"
-					(reference "J16")
+					(reference "J3")
 					(unit 1)
 				)
@@
 		(on_board yes)
 		(dnp no)
-		(property "Reference" "R30"
+		(property "Reference" "R32"
 			(at 51.435 106.045 90)
 			(effects
@@
 			(project ""
 				(path "/2eea20e6-112c-411a-b615-885ae773135a/00000000-0000-0000-0000-000061bef9ce"
-					(reference "R30")
+					(reference "R32")
 					(unit 1)
 				)
@@
 		(dnp no)
 		(fields_autoplaced yes)
-		(property "Reference" "J14"
+		(property "Reference" "J15"
 			(at 196.85 44.4499 0)
 			(effects
@@
 			(project ""
 				(path "/2eea20e6-112c-411a-b615-885ae773135a/00000000-0000-0000-0000-000061bef9ce"
-					(reference "J14")
+					(reference "J15")
 					(unit 1)
 				)
@@
 		(on_board yes)
 		(dnp no)
-		(property "Reference" "JP6"
+		(property "Reference" "JP5"
 			(at 130.81 49.53 0)
 			(effects
@@
 			(project ""
 				(path "/2eea20e6-112c-411a-b615-885ae773135a/00000000-0000-0000-0000-000061bef9ce"
-					(reference "JP6")
+					(reference "JP5")
 					(unit 1)
 				)
@@
 		(on_board yes)
 		(dnp no)
-		(property "Reference" "JP2"
+		(property "Reference" "JP1"
 			(at 54.61 88.9 0)
 			(effects
@@
 			(project ""
 				(path "/2eea20e6-112c-411a-b615-885ae773135a/00000000-0000-0000-0000-000061bef9ce"
-					(reference "JP2")
+					(reference "JP1")
 					(unit 1)
 				)
@@
 		(on_board yes)
 		(dnp no)
-		(property "Reference" "R32"
+		(property "Reference" "R34"
 			(at 197.0786 95.3516 0)
 			(effects
@@
 			(project ""
 				(path "/2eea20e6-112c-411a-b615-885ae773135a/00000000-0000-0000-0000-000061bef9ce"
-					(reference "R32")
+					(reference "R34")
 					(unit 1)
 				)
@@
 		(on_board yes)
 		(dnp no)
-		(property "Reference" "JP4"
+		(property "Reference" "JP3"
 			(at 92.71 69.85 0)
 			(effects
@@
 			(project ""
 				(path "/2eea20e6-112c-411a-b615-885ae773135a/00000000-0000-0000-0000-000061bef9ce"
-					(reference "JP4")
+					(reference "JP3")
 					(unit 1)
 				)
@@
 		(on_board yes)
 		(dnp no)
-		(property "Reference" "C76"
+		(property "Reference" "C77"
 			(at 36.6268 176.4284 0)
 			(effects
@@
 			(project ""
 				(path "/2eea20e6-112c-411a-b615-885ae773135a/00000000-0000-0000-0000-000061bef9ce"
-					(reference "C76")
+					(reference "C77")
 					(unit 1)
 				)
@@
 		(on_board yes)
 		(dnp no)
-		(property "Reference" "JP3"
+		(property "Reference" "JP2"
 			(at 74.93 88.9 0)
 			(effects
@@
 			(project ""
 				(path "/2eea20e6-112c-411a-b615-885ae773135a/00000000-0000-0000-0000-000061bef9ce"
-					(reference "JP3")
+					(reference "JP2")
 					(unit 1)
 				)
@@
 		(dnp no)
 		(fields_autoplaced yes)
-		(property "Reference" "J15"
+		(property "Reference" "J16"
 			(at 242.57 44.4499 0)
 			(effects
@@
 			(project ""
 				(path "/2eea20e6-112c-411a-b615-885ae773135a/00000000-0000-0000-0000-000061bef9ce"
-					(reference "J15")
+					(reference "J16")
 					(unit 1)
 				)
@@
 		(on_board yes)
 		(dnp no)
-		(property "Reference" "R33"
+		(property "Reference" "R35"
 			(at 197.0786 137.2616 0)
 			(effects
@@
 			(project ""
 				(path "/2eea20e6-112c-411a-b615-885ae773135a/00000000-0000-0000-0000-000061bef9ce"
-					(reference "R33")
+					(reference "R35")
 					(unit 1)
 				)
@@
 		(on_board yes)
 		(dnp no)
-		(property "Reference" "JP7"
+		(property "Reference" "JP6"
 			(at 151.13 49.53 0)
 			(effects
@@
 			(project ""
 				(path "/2eea20e6-112c-411a-b615-885ae773135a/00000000-0000-0000-0000-000061bef9ce"
-					(reference "JP7")
+					(reference "JP6")
 					(unit 1)
 				)
@@
 		(on_board yes)
 		(dnp no)
-		(property "Reference" "R31"
+		(property "Reference" "R33"
 			(at 51.435 111.125 90)
 			(effects
@@
 			(project ""
 				(path "/2eea20e6-112c-411a-b615-885ae773135a/00000000-0000-0000-0000-000061bef9ce"
-					(reference "R31")
+					(reference "R33")
 					(unit 1)
 				)
@@
 		(on_board yes)
 		(dnp no)
-		(property "Reference" "JP5"
+		(property "Reference" "JP4"
 			(at 113.03 69.85 0)
 			(effects
@@
 			(project ""
 				(path "/2eea20e6-112c-411a-b615-885ae773135a/00000000-0000-0000-0000-000061bef9ce"
-					(reference "JP5")
-					(unit 1)
-				)
+					(reference "JP4")
+					(unit 1)
+				)

Commit message: hw: tidy warnings
Parts:
- J3, J6: footprint Retrocomputing:CBM_PET_CASS_EDGE_CON_12P -> EconoPET:CBM_PET_CASS_EDGE_CON_12P
Changed lines of the file:
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@@
 			)
 		)
-		(property "Footprint" "Retrocomputing:CBM_PET_CASS_EDGE_CON_12P"
+		(property "Footprint" "EconoPET:CBM_PET_CASS_EDGE_CON_12P"
 			(at 243.84 154.94 0)
 			(effects
@@
 			)
 		)
-		(property "Footprint" "Retrocomputing:CBM_PET_CASS_EDGE_CON_12P"
+		(property "Footprint" "EconoPET:CBM_PET_CASS_EDGE_CON_12P"
 			(at 243.84 113.03 0)
 			(effects
