File: hw/rev-c/mainboard/kicad/USER.kicad_sch (KiCad schematic)
At the start: 4 parts, among them J16 USER_HEADER, J2 USER

Commit message: hw: fix wire/grid violations in schematic
Parts:
- J2: symbol Retrocomputing:CBM_PET_USER_Conn_02x12_Card_Edge -> EconoPET:CBM_PET_USER_Conn_02x12_Card_Edge
Changed lines of the file:
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@@
 	)
 	(symbol
-		(lib_id "Retrocomputing:CBM_PET_USER_Conn_02x12_Card_Edge")
+		(lib_id "EconoPET:CBM_PET_USER_Conn_02x12_Card_Edge")
 		(at 106.68 93.98 0)
 		(unit 1)

Commit message: hw: renumber reference designators
Parts:
- renumbered C104 to C75, J2 to J12, J16 to J13
Changed lines of the file:
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@@
 		(on_board yes)
 		(dnp no)
-		(property "Reference" "J2"
+		(property "Reference" "J12"
 			(at 107.95 75.7682 0)
 			(effects
@@
 			(project ""
 				(path "/2eea20e6-112c-411a-b615-885ae773135a/00000000-0000-0000-0000-000061b3f8ab"
-					(reference "J2")
+					(reference "J12")
 					(unit 1)
 				)
@@
 		(dnp no)
 		(fields_autoplaced yes)
-		(property "Reference" "J16"
+		(property "Reference" "J13"
 			(at 177.8 76.2 0)
 			(effects
@@
 			(project ""
 				(path "/2eea20e6-112c-411a-b615-885ae773135a/00000000-0000-0000-0000-000061b3f8ab"
-					(reference "J16")
+					(reference "J13")
 					(unit 1)
 				)
@@
 		(on_board yes)
 		(dnp no)
-		(property "Reference" "C104"
+		(property "Reference" "C75"
 			(at 201.7268 110.5916 0)
 			(effects
@@
 			(project ""
 				(path "/2eea20e6-112c-411a-b615-885ae773135a/00000000-0000-0000-0000-000061b3f8ab"
-					(reference "C104")
+					(reference "C75")
 					(unit 1)
 				)

Commit message: hw: header for 5v/video select, ESR for AMS1117 + tidy
Parts:
- removed JP1: VIDEO_OR_5V, Jumper:SolderJumper-3_P1.3mm_Bridged12_RoundedPad1.0x1.5mm, symbol Jumper:SolderJumper_3_Open
- added J26: VIDEO_OR_5V, Connector_PinHeader_2.54mm:PinHeader_1x03_P2.54mm_Vertical, symbol Connector:Conn_01x03_Pin
Connections:
- net +5V: now also J26.3 (Pin_3)
- net BVIDEO: now also J26.1 (Pin_1)
- net VIDEO_OR_5V: now also J26.2 (Pin_2)
Other:
- moved on the sheet: C75, J12, J13

Commit message: hw: match original PET designators for connectors
Parts:
- J12: renamed from J26; footprint Connector_PinHeader_2.54mm:PinHeader_1x03_P2.54mm_Vertical -> EconoPET:PinHeader_1x03_P2.54mm_Vertical_or_SolderJumper
- renumbered C75 to C76, J13 to J14, J12 to J2
Changed lines of the file:
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@@
 		(on_board yes)
 		(dnp no)
-		(property "Reference" "J12"
+		(property "Reference" "J2"
 			(at 124.46 82.1182 0)
 			(effects
@@
 			(project ""
 				(path "/2eea20e6-112c-411a-b615-885ae773135a/00000000-0000-0000-0000-000061b3f8ab"
-					(reference "J12")
+					(reference "J2")
 					(unit 1)
 				)
@@
 		(dnp no)
 		(fields_autoplaced yes)
-		(property "Reference" "J13"
+		(property "Reference" "J14"
 			(at 194.31 82.55 0)
 			(effects
@@
 			(project ""
 				(path "/2eea20e6-112c-411a-b615-885ae773135a/00000000-0000-0000-0000-000061b3f8ab"
-					(reference "J13")
+					(reference "J14")
 					(unit 1)
 				)
@@
 		(on_board yes)
 		(dnp no)
-		(property "Reference" "C75"
+		(property "Reference" "C76"
 			(at 218.2368 116.9416 0)
 			(effects
@@
 			(project ""
 				(path "/2eea20e6-112c-411a-b615-885ae773135a/00000000-0000-0000-0000-000061b3f8ab"
-					(reference "C75")
+					(reference "C76")
 					(unit 1)
 				)
@@
 		(on_board yes)
 		(dnp no)
-		(property "Reference" "J26"
+		(property "Reference" "J12"
 			(at 73.152 75.438 0)
 			(effects
@@
 			)
 		)
-		(property "Footprint" "Connector_PinHeader_2.54mm:PinHeader_1x03_P2.54mm_Vertical"
+		(property "Footprint" "EconoPET:PinHeader_1x03_P2.54mm_Vertical_or_SolderJumper"
 			(at 76.2 83.82 0)
 			(effects
@@
 			(project ""
 				(path "/2eea20e6-112c-411a-b615-885ae773135a/00000000-0000-0000-0000-000061b3f8ab"
-					(reference "J26")
-					(unit 1)
-				)
+					(reference "J12")
+					(unit 1)
+				)

Commit message: hw: tidy warnings
Parts:
- J2: footprint Retrocomputing:CBM_PET_USER_EDGE_CON_24P -> EconoPET:CBM_PET_USER_EDGE_CON_24P
Changed lines of the file:
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@@
 			)
 		)
-		(property "Footprint" "Retrocomputing:CBM_PET_USER_EDGE_CON_24P"
+		(property "Footprint" "EconoPET:CBM_PET_USER_EDGE_CON_24P"
 			(at 123.19 100.33 0)
 			(effects

Commit message: hw: routing touchups, killer poke mitigation
Parts:
- C76: value 4.7u 10V -> 4u7; LCSC C23733 -> C1538
Changed lines of the file:
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@@
 			)
 		)
-		(property "Value" "4.7u 10V"
+		(property "Value" "4u7"
 			(at 218.2368 119.253 0)
 			(effects
@@
 			)
 		)
-		(property "Datasheet" "https://product.samsungsem.com/mlcc/CL05A475MP5NRN.do"
+		(property "Datasheet" "https://www.lcsc.com/datasheet/lcsc_datasheet_2304140030_FH--Guangdong-Fenghua-Advanced-Tech-0402B472K500NT_C1538.pdf"
 			(at 215.9 118.11 0)
 			(effects
@@
 			)
 		)
-		(property "LCSC" "C23733"
+		(property "LCSC" "C1538"
 			(at 215.9 118.11 0)
 			(effects
