File: hw/rev-c/mainboard/kicad/FLASH.kicad_sch (KiCad schematic)
At the start: 5 parts, among them SW6 BOOTSEL, U22 W25Q128JVS

Commit message: hw: renumber reference designators
Parts:
- renumbered C102 to C103, R58 to R63, R59 to R64

Commit message: hw: match original PET designators for connectors
Parts:
- renumbered C103 to C104, R63 to R65, R64 to R66
Changed lines of the file:
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@@
 		(on_board yes)
 		(dnp no)
-		(property "Reference" "R64"
+		(property "Reference" "R66"
 			(at 121.285 90.805 90)
 			(effects
@@
 			(project ""
 				(path "/2eea20e6-112c-411a-b615-885ae773135a/00000000-0000-0000-0000-0000617d6918/b70241ab-8a5c-42d5-a1ab-8f4bc50a1197/3b6d0c70-6282-4619-97c5-f97c852cfe84"
-					(reference "R64")
+					(reference "R66")
 					(unit 1)
 				)
@@
 		(on_board yes)
 		(dnp no)
-		(property "Reference" "R63"
+		(property "Reference" "R65"
 			(at 111.125 97.155 90)
 			(effects
@@
 			(project ""
 				(path "/2eea20e6-112c-411a-b615-885ae773135a/00000000-0000-0000-0000-0000617d6918/b70241ab-8a5c-42d5-a1ab-8f4bc50a1197/3b6d0c70-6282-4619-97c5-f97c852cfe84"
-					(reference "R63")
+					(reference "R65")
 					(unit 1)
 				)
@@
 		(on_board yes)
 		(dnp no)
-		(property "Reference" "C103"
+		(property "Reference" "C104"
 			(at 148.3868 77.5716 0)
 			(effects
@@
 			(project ""
 				(path "/2eea20e6-112c-411a-b615-885ae773135a/00000000-0000-0000-0000-0000617d6918/b70241ab-8a5c-42d5-a1ab-8f4bc50a1197/3b6d0c70-6282-4619-97c5-f97c852cfe84"
-					(reference "C103")
-					(unit 1)
-				)
+					(reference "C104")
+					(unit 1)
+				)

Commit message: hw: tidy warnings
Parts:
- SW6: footprint JLCPCB:SW-TH_L6.0-W3.5-P6.50 -> EconoPET:SW_PUSH_1P1T_6x3.5mm_H4.3_APEM_MJTP1243
- U22: footprint Package_SO:SOIC-8_5.23x5.23mm_P1.27mm -> EconoPET:SOIC-8_5.23x5.23mm_P1.27mm
- renumbered C104 to C1
Changed lines of the file:
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@@
 			)
 		)
-		(property "Footprint" "JLCPCB:SW-TH_L6.0-W3.5-P6.50"
+		(property "Footprint" "EconoPET:SW_PUSH_1P1T_6x3.5mm_H4.3_APEM_MJTP1243"
 			(at 107.95 107.95 0)
 			(effects
@@
 		(on_board yes)
 		(dnp no)
-		(property "Reference" "C104"
+		(property "Reference" "C1"
 			(at 148.3868 77.5716 0)
 			(effects
@@
 			(project ""
 				(path "/2eea20e6-112c-411a-b615-885ae773135a/00000000-0000-0000-0000-0000617d6918/b70241ab-8a5c-42d5-a1ab-8f4bc50a1197/3b6d0c70-6282-4619-97c5-f97c852cfe84"
-					(reference "C104")
+					(reference "C1")
 					(unit 1)
 				)
@@
 			)
 		)
-		(property "Footprint" "Package_SO:SOIC-8_5.23x5.23mm_P1.27mm"
+		(property "Footprint" "EconoPET:SOIC-8_5.23x5.23mm_P1.27mm"
 			(at 142.24 101.6 0)
 			(effects
