File: hw/rev-c/mainboard/kicad/IO.kicad_sch (KiCad schematic)
At the start: 6 parts, among them U11 W65C21N, U12 W65C21N, U13 W65C22N

Commit message: hw: fix wire/grid violations in schematic
Parts:
- U11, U12: symbol Mainboard-rescue:W65C21NxP-PET -> EconoPET:W65C21N
- U13: symbol Mainboard-rescue:W65C22NxP-PET -> EconoPET:W65C22N
Changed lines of the file:
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@@
 	)
 	(symbol
-		(lib_id "Mainboard-rescue:W65C21NxP-PET")
+		(lib_id "EconoPET:W65C21N")
 		(at 86.36 153.67 0)
 		(unit 1)
@@
 	)
 	(symbol
-		(lib_id "Mainboard-rescue:W65C22NxP-PET")
+		(lib_id "EconoPET:W65C22N")
 		(at 184.15 128.27 0)
 		(unit 1)
@@
 	)
 	(symbol
-		(lib_id "Mainboard-rescue:W65C21NxP-PET")
+		(lib_id "EconoPET:W65C21N")
 		(at 86.36 58.42 0)
 		(unit 1)

Commit message: hw: match original PET designators for connectors
Parts:
- renumbered C66 to C67, C67 to C68, C68 to C69
Changed lines of the file:
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@@
 		(on_board yes)
 		(dnp no)
-		(property "Reference" "C66"
+		(property "Reference" "C67"
 			(at 97.79 111.76 90)
 			(effects
@@
 			(project ""
 				(path "/2eea20e6-112c-411a-b615-885ae773135a/00000000-0000-0000-0000-000061b9c2eb"
-					(reference "C66")
+					(reference "C67")
 					(unit 1)
 				)
@@
 		(on_board yes)
 		(dnp no)
-		(property "Reference" "C67"
+		(property "Reference" "C68"
 			(at 101.6 16.51 90)
 			(effects
@@
 			(project ""
 				(path "/2eea20e6-112c-411a-b615-885ae773135a/00000000-0000-0000-0000-000061b9c2eb"
-					(reference "C67")
+					(reference "C68")
 					(unit 1)
 				)
@@
 		(on_board yes)
 		(dnp no)
-		(property "Reference" "C68"
+		(property "Reference" "C69"
 			(at 198.12 85.09 90)
 			(effects
@@
 			(project ""
 				(path "/2eea20e6-112c-411a-b615-885ae773135a/00000000-0000-0000-0000-000061b9c2eb"
-					(reference "C68")
+					(reference "C69")
 					(unit 1)
 				)

Commit message: hw: routing touchups, killer poke mitigation
Parts:
- added R38: 470, Resistor_SMD:R_0402_1005Metric, symbol Device:R_Small
Connections:
- net BVERT: now also R38.2; no longer U13.15 (PB5)
- new net: R38.1, U13.15 (PB5)
Other:
- note added: "470R mitigates "killer poke", which configures PB5 as an output. W65C22N drives 1 CMOS load (or two TTL loads). BVERT is driven high/low at +/- 24ma by SN74LVC4245APWR."
- note added: "Signals with a 'B' prefix have been level shifted from 3V3 to 5V Note that ~{IRQ} is wire-or'ed and pulled to 3V3 (not 5V)"
- note removed: "Signals with a 'B' prefix have been level shifted from 3V3 to 5V ~{IRQ} is wire-or'ed and pulled to 3V3 (not 5V)"
Changed lines of the file:
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@@
 	(wire
 		(pts
-			(xy 199.39 143.51) (xy 234.95 143.51)
-		)
-		(stroke
-			(width 0)
-			(type default)
-		)
-	)
-	(wire
-		(pts
 			(xy 55.88 78.74) (xy 71.12 78.74)
 		)
@@
 	(wire
 		(pts
+			(xy 199.39 143.51) (xy 222.25 143.51)
+		)
+		(stroke
+			(width 0)
+			(type default)
+		)
+	)
+	(wire
+		(pts
 			(xy 111.76 73.66) (xy 101.6 73.66)
 		)
@@
 	(wire
 		(pts
+			(xy 227.33 143.51) (xy 234.95 143.51)
+		)
+		(stroke
+			(width 0)
+			(type default)
+		)
+	)
+	(wire
+		(pts
 			(xy 101.6 118.11) (xy 100.33 118.11)
 		)
@@
 		)
 	)
+	(text "470R mitigates \"killer poke\",\nwhich configures PB5 as an output.\n\nW65C22N drives 1 CMOS load\n(or two TTL loads).\n\nBVERT is driven high/low at\n+/- 24ma by SN74LVC4245APWR."
+		(exclude_from_sim no)
+		(at 220.472 159.258 0)
+		(effects
+			(font
+				(size 1.27 1.27)
+			)
+			(justify left)
+		)
+	)
 	(text "PIA1"
 		(exclude_from_sim no)
@@
 		)
 	)
-	(text "Signals with a 'B' prefix have been level shifted from 3V3 to 5V\n\n~{IRQ} is wire-or'ed and pulled to 3V3 (not 5V)"
+	(text "Signals with a 'B' prefix have been level shifted from 3V3 to 5V\n\nNote that ~{IRQ} is wire-or'ed and pulled to 3V3 (not 5V)"
 		(exclude_from_sim no)
 		(at 146.05 46.99 0)
@@
 		)
 	)
+	(label "BVERT"
+		(at 228.6 143.51 0)
+		(fields_autoplaced yes)
+		(effects
+			(font
+				(size 1.27 1.27)
+			)
+			(justify left bottom)
+		)
+	)
 	(label "BD4"
 		(at 168.91 148.59 180)
@@
 					(unit 1)
 				)
+			)
+		)
+	)
+	(symbol
+		(lib_id "Device:R_Small")
+		(at 224.79 143.51 90)
+		(mirror x)
+		(unit 1)
+		(exclude_from_sim no)
+		(in_bom yes)
+		(on_board yes)
+		(dnp no)
+		(property "Reference" "R38"
+			(at 226.822 146.05 90)
+			(effects
+				(font
+					(size 1.27 1.27)
+				)
+				(justify left)
+			)
+		)
+		(property "Value" "470"
+			(at 226.822 148.082 90)
+			(effects
+				(font
+					(size 1.27 1.27)
+				)
+				(justify left)
+			)
+		)
+		(property "Footprint" "Resistor_SMD:R_0402_1005Metric"
+			(at 224.79 143.51 0)
+			(effects
+				(font
+					(size 1.27 1.27)
+				)
+				(hide yes)
+			)
+		)
+		(property "Datasheet" "https://datasheet.lcsc.com/lcsc/2205311900_UNI-ROYAL-Uniroyal-Elec-0402WGF4700TCE_C25117.pdf"
+			(at 224.79 143.51 0)
+			(effects
+				(font
+					(size 1.27 1.27)
+				)
+				(hide yes)
+			)
+		)
+		(property "Description" ""
+			(at 224.79 143.51 0)
+			(effects
+				(font
+					(size 1.27 1.27)
+				)
+				(hide yes)
+			)
+		)
+		(property "LCSC" "C25117"
+			(at 224.79 143.51 0)
+			(effects
+				(font
+					(size 1.27 1.27)
+				)
+				(hide yes)
+			)
+		)
+		(pin "1"
+		)
+		(pin "2"
+		)
+		(instances
+			(project "Mainboard"
+				(path "/2eea20e6-112c-411a-b615-885ae773135a/00000000-0000-0000-0000-000061b9c2eb"
+					(reference "R38")
+					(unit 1)
+				)

Commit message: hw: tidy
Other:
- note added: ""Killer Poke" puts PB5 in contention with BVERT. W65C22N drives 1 CMOS load (~3ma). BVERT is driven at ~24ma by level shifter. I_{MAX} is ~20ma per pin CMOS, ~16ma TTL? CMOS rule of thumb is 220-1K Ω. 470Ω passes ~10ma, which is further reduced by built-in series resistors in the W65C22N."
- note removed: "470R mitigates "killer poke", which configures PB5 as an output. W65C22N drives 1 CMOS load (or two TTL loads). BVERT is driven high/low at +/- 24ma by SN74LVC4245APWR."
- moved on the sheet: R38
Changed lines of the file:
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@@
 	(wire
 		(pts
-			(xy 199.39 143.51) (xy 222.25 143.51)
+			(xy 199.39 143.51) (xy 224.79 143.51)
 		)
 		(stroke
@@
 	(wire
 		(pts
-			(xy 227.33 143.51) (xy 234.95 143.51)
+			(xy 229.87 143.51) (xy 234.95 143.51)
 		)
 		(stroke
@@
 		)
 	)
-	(text "470R mitigates \"killer poke\",\nwhich configures PB5 as an output.\n\nW65C22N drives 1 CMOS load\n(or two TTL loads).\n\nBVERT is driven high/low at\n+/- 24ma by SN74LVC4245APWR."
+	(text "\"Killer Poke\" puts PB5 in contention with BVERT.\n\nW65C22N drives 1 CMOS load (~3ma).\nBVERT is driven at ~24ma by level shifter.\nI_{MAX} is ~20ma per pin CMOS, ~16ma TTL?\nCMOS rule of thumb is 220-1K Ω.\n470Ω passes ~10ma, which is further reduced\nby built-in series resistors in the W65C22N."
 		(exclude_from_sim no)
-		(at 220.472 159.258 0)
+		(at 217.678 155.702 0)
 		(effects
 			(font
@@
 	(label "DIO_IN4"
 		(at 101.6 133.35 0)
-		(fields_autoplaced yes)
-		(effects
-			(font
-				(size 1.27 1.27)
-			)
-			(justify left bottom)
-		)
-	)
-	(label "BVERT"
-		(at 228.6 143.51 0)
 		(fields_autoplaced yes)
 		(effects
@@
 		(dnp no)
 		(property "Reference" "C67"
-			(at 97.79 111.76 90)
+			(at 99.06 111.76 90)
 			(effects
 				(font
@@
 		(dnp no)
 		(property "Reference" "C69"
-			(at 198.12 85.09 90)
+			(at 199.39 85.09 90)
 			(effects
 				(font
@@
 	(symbol
 		(lib_id "Device:R_Small")
-		(at 224.79 143.51 90)
+		(at 227.33 143.51 90)
 		(mirror x)
 		(unit 1)
@@
 		(dnp no)
 		(property "Reference" "R38"
-			(at 226.822 146.05 90)
+			(at 229.108 138.43 90)
 			(effects
 				(font
@@
 		)
 		(property "Value" "470"
-			(at 226.822 148.082 90)
+			(at 229.108 140.462 90)
 			(effects
 				(font
@@
 		)
 		(property "Footprint" "Resistor_SMD:R_0402_1005Metric"
-			(at 224.79 143.51 0)
+			(at 227.33 143.51 0)
 			(effects
 				(font
@@
 			)
 		)
-		(property "Datasheet" "https://datasheet.lcsc.com/lcsc/2205311900_UNI-ROYAL-Uniroyal-Elec-0402WGF4700TCE_C25117.pdf"
-			(at 224.79 143.51 0)
+		(property "Datasheet" ""
+			(at 227.33 143.51 0)
 			(effects
 				(font
@@
 		)
 		(property "Description" ""
-			(at 224.79 143.51 0)
+			(at 227.33 143.51 0)
 			(effects
 				(font
@@
 		)
 		(property "LCSC" "C25117"
-			(at 224.79 143.51 0)
-			(effects
-				(font
+			(at 227.33 143.51 0)
+			(effects
+				(font
