File: hw/rev-c/mainboard/kicad/MicroSD.kicad_sch (KiCad schematic)
At the start: 5 parts, among them J23 MICRO_SD

Commit message: hw: update uSD symbol/footprint
Parts:
- J23: symbol Connector:Micro_SD_Card_Det -> Connector:Micro_SD_Card_Det1
Connections:
- net GND: no longer J23.11 (SHIELD), J23.12 (SHIELD), J23.13 (SHIELD)
Changed lines of the file:
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@@
 	)
 	(symbol
-		(lib_id "Connector:Micro_SD_Card_Det")
+		(lib_id "Connector:Micro_SD_Card_Det1")
 		(at 172.72 99.06 0)
 		(unit 1)
@@
 			)
 		)
-		(property "Description" ""
+		(property "Description" "Micro SD Card Socket with one card detection pin"
 			(at 172.72 99.06 0)
 			(effects
@@
 			)
 		)
-		(pin "11"
-		)
-		(pin "12"
-		)
-		(pin "13"
-		)
 		(pin "1"

Commit message: hw: renumber reference designators
Parts:
- renumbered C99 to C100, C98 to C99, J23 to J24, R55 to R60
Changed lines of the file:
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@@
 		(on_board yes)
 		(dnp no)
-		(property "Reference" "#PWR0165"
+		(property "Reference" "#PWR0166"
 			(at 138.43 78.74 0)
 			(effects
@@
 			(project ""
 				(path "/2eea20e6-112c-411a-b615-885ae773135a/00000000-0000-0000-0000-0000617d6918/b70241ab-8a5c-42d5-a1ab-8f4bc50a1197/d7346628-bc14-4709-aafe-5231479d808e"
-					(reference "#PWR0165")
+					(reference "#PWR0166")
 					(unit 1)
 				)
@@
 		(on_board yes)
 		(dnp no)
-		(property "Reference" "#PWR0166"
+		(property "Reference" "#PWR0167"
 			(at 147.32 68.58 0)
 			(effects
@@
 			(project ""
 				(path "/2eea20e6-112c-411a-b615-885ae773135a/00000000-0000-0000-0000-0000617d6918/b70241ab-8a5c-42d5-a1ab-8f4bc50a1197/d7346628-bc14-4709-aafe-5231479d808e"
-					(reference "#PWR0166")
+					(reference "#PWR0167")
 					(unit 1)
 				)
@@
 		(dnp no)
 		(fields_autoplaced yes)
-		(property "Reference" "J23"
+		(property "Reference" "J24"
 			(at 173.355 77.47 0)
 			(effects
@@
 			(project ""
 				(path "/2eea20e6-112c-411a-b615-885ae773135a/00000000-0000-0000-0000-0000617d6918/b70241ab-8a5c-42d5-a1ab-8f4bc50a1197/d7346628-bc14-4709-aafe-5231479d808e"
-					(reference "J23")
+					(reference "J24")
 					(unit 1)
 				)
@@
 		(dnp no)
 		(fields_autoplaced yes)
-		(property "Reference" "#PWR0169"
+		(property "Reference" "#PWR0170"
 			(at 194.31 119.38 0)
 			(effects
@@
 			(project ""
 				(path "/2eea20e6-112c-411a-b615-885ae773135a/00000000-0000-0000-0000-0000617d6918/b70241ab-8a5c-42d5-a1ab-8f4bc50a1197/d7346628-bc14-4709-aafe-5231479d808e"
-					(reference "#PWR0169")
+					(reference "#PWR0170")
 					(unit 1)
 				)
@@
 		(dnp no)
 		(fields_autoplaced yes)
-		(property "Reference" "#PWR0167"
+		(property "Reference" "#PWR0168"
 			(at 147.32 124.46 0)
 			(effects
@@
 			(project ""
 				(path "/2eea20e6-112c-411a-b615-885ae773135a/00000000-0000-0000-0000-0000617d6918/b70241ab-8a5c-42d5-a1ab-8f4bc50a1197/d7346628-bc14-4709-aafe-5231479d808e"
-					(reference "#PWR0167")
+					(reference "#PWR0168")
 					(unit 1)
 				)
@@
 		(on_board yes)
 		(dnp no)
-		(property "Reference" "R55"
+		(property "Reference" "R60"
 			(at 118.745 83.185 90)
 			(effects
@@
 			(project ""
 				(path "/2eea20e6-112c-411a-b615-885ae773135a/00000000-0000-0000-0000-0000617d6918/b70241ab-8a5c-42d5-a1ab-8f4bc50a1197/d7346628-bc14-4709-aafe-5231479d808e"
-					(reference "R55")
+					(reference "R60")
 					(unit 1)
 				)
@@
 		(dnp no)
 		(fields_autoplaced yes)
-		(property "Reference" "#PWR0168"
+		(property "Reference" "#PWR0169"
 			(at 154.94 81.28 0)
 			(effects
@@
 			(project ""
 				(path "/2eea20e6-112c-411a-b615-885ae773135a/00000000-0000-0000-0000-0000617d6918/b70241ab-8a5c-42d5-a1ab-8f4bc50a1197/d7346628-bc14-4709-aafe-5231479d808e"
-					(reference "#PWR0168")
+					(reference "#PWR0169")
 					(unit 1)
 				)
@@
 		(on_board yes)
 		(dnp no)
-		(property "Reference" "C99"
+		(property "Reference" "C100"
 			(at 167.4368 68.6816 0)
 			(effects
@@
 			(project ""
 				(path "/2eea20e6-112c-411a-b615-885ae773135a/00000000-0000-0000-0000-0000617d6918/b70241ab-8a5c-42d5-a1ab-8f4bc50a1197/d7346628-bc14-4709-aafe-5231479d808e"
-					(reference "C99")
+					(reference "C100")
 					(unit 1)
 				)
@@
 		(on_board yes)
 		(dnp no)
-		(property "Reference" "C98"
+		(property "Reference" "C99"
 			(at 157.2768 68.6816 0)
 			(effects
@@
 			(project ""
 				(path "/2eea20e6-112c-411a-b615-885ae773135a/00000000-0000-0000-0000-0000617d6918/b70241ab-8a5c-42d5-a1ab-8f4bc50a1197/d7346628-bc14-4709-aafe-5231479d808e"
-					(reference "C98")
-					(unit 1)
-				)
+					(reference "C99")
+					(unit 1)
+				)

Commit message: hw: match original PET designators for connectors
Parts:
- renumbered C99 to C100, C100 to C101, J24 to J25, R60 to R62
Changed lines of the file:
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@@
 		(dnp no)
 		(fields_autoplaced yes)
-		(property "Reference" "J24"
+		(property "Reference" "J25"
 			(at 173.355 77.47 0)
 			(effects
@@
 			(project ""
 				(path "/2eea20e6-112c-411a-b615-885ae773135a/00000000-0000-0000-0000-0000617d6918/b70241ab-8a5c-42d5-a1ab-8f4bc50a1197/d7346628-bc14-4709-aafe-5231479d808e"
-					(reference "J24")
+					(reference "J25")
 					(unit 1)
 				)
@@
 		(on_board yes)
 		(dnp no)
-		(property "Reference" "R60"
+		(property "Reference" "R62"
 			(at 118.745 83.185 90)
 			(effects
@@
 			(project ""
 				(path "/2eea20e6-112c-411a-b615-885ae773135a/00000000-0000-0000-0000-0000617d6918/b70241ab-8a5c-42d5-a1ab-8f4bc50a1197/d7346628-bc14-4709-aafe-5231479d808e"
-					(reference "R60")
+					(reference "R62")
 					(unit 1)
 				)
@@
 		(on_board yes)
 		(dnp no)
-		(property "Reference" "C100"
+		(property "Reference" "C101"
 			(at 167.4368 68.6816 0)
 			(effects
@@
 			(project ""
 				(path "/2eea20e6-112c-411a-b615-885ae773135a/00000000-0000-0000-0000-0000617d6918/b70241ab-8a5c-42d5-a1ab-8f4bc50a1197/d7346628-bc14-4709-aafe-5231479d808e"
-					(reference "C100")
+					(reference "C101")
 					(unit 1)
 				)
@@
 		(on_board yes)
 		(dnp no)
-		(property "Reference" "C99"
+		(property "Reference" "C100"
 			(at 157.2768 68.6816 0)
 			(effects
@@
 			(project ""
 				(path "/2eea20e6-112c-411a-b615-885ae773135a/00000000-0000-0000-0000-0000617d6918/b70241ab-8a5c-42d5-a1ab-8f4bc50a1197/d7346628-bc14-4709-aafe-5231479d808e"
-					(reference "C99")
-					(unit 1)
-				)
+					(reference "C100")
+					(unit 1)
+				)

Commit message: hw: tidy warnings
Parts:
- renumbered C100 to C2
Changed lines of the file:
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@@
 		(on_board yes)
 		(dnp no)
-		(property "Reference" "C100"
+		(property "Reference" "C2"
 			(at 157.2768 68.6816 0)
 			(effects
@@
 			(project ""
 				(path "/2eea20e6-112c-411a-b615-885ae773135a/00000000-0000-0000-0000-0000617d6918/b70241ab-8a5c-42d5-a1ab-8f4bc50a1197/d7346628-bc14-4709-aafe-5231479d808e"
-					(reference "C100")
+					(reference "C2")
 					(unit 1)
 				)

Commit message: hw: fix/update parts / use parallel resistors to control 5V
Parts:
- RN16: value 10k -> 10kx4
Changed lines of the file:
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@@
 			)
 		)
-		(property "Datasheet" "https://datasheet.lcsc.com/lcsc/1912111437_SHOU-HAN-TF-PUSH_C393941.pdf"
+		(property "Datasheet" "https://www.lcsc.com/datasheet/lcsc_datasheet_1912111437_SHOU-HAN-TF-PUSH_C393941.pdf"
 			(at 172.72 118.11 0)
 			(effects
@@
 			)
 		)
-		(property "Value" "10k"
+		(property "Value" "10kx4"
 			(at 128.905 82.55 0)
 			(effects
@@
 			)
 		)
-		(property "Datasheet" "https://datasheet.lcsc.com/lcsc/2304140030_UNI-ROYAL-Uniroyal-Elec-4D03WGJ0103T5E_C29718.pdf"
+		(property "Datasheet" "https://www.lcsc.com/datasheet/lcsc_datasheet_2304140030_UNI-ROYAL-Uniroyal-Elec-4D03WGJ0103T5E_C29718.pdf"
 			(at 133.35 81.28 0)
 			(effects
@@
 			)
 		)
-		(property "Datasheet" "https://datasheet.lcsc.com/lcsc/2206010100_UNI-ROYAL-Uniroyal-Elec-0402WGF1002TCE_C25744.pdf"
+		(property "Datasheet" "https://jlcpcb.com/api/file/downloadByFileSystemAccessId/8556212101498380288"
 			(at 120.65 81.28 0)
 			(effects
@@
 			)
 		)
-		(property "Datasheet" "https://datasheet.lcsc.com/lcsc/2304140030_Samsung-Electro-Mechanics-CL05B104KB54PNC_C307331.pdf"
+		(property "Datasheet" "https://product.samsungsem.com/mlcc/CL05B104KB54PN.do"
 			(at 154.94 69.85 0)
 			(effects
