File: hw/rev-a/mainboard/kicad/Audio.kicad_sch (KiCad schematic)
At the start: 27 parts, among them J21 AUDIO, Q4 SS8050, Q5 SS8050, Q6 SS8050, Q7 SS8550

Commit message: hw: tidy schematics for publication
Other:
- note added: "Audio"
- note added: "PET CB2 and DIAG are inputs to FPGA. FPGA implements AND gate and outputs AUDIO source. This saves an IC and allows for experimental enhancements, like SID emulation at $8F00. The AUDIO source is ΔΣ encoded 1-bit output from the FPGA (3V3 at 64 MHz). The 1u capacitor and 12k resistor adjusts this to line-level audio, which is +/- 0.5V AC for consumer electronics. (Note that amplifiers and powered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"
- note removed: "The AUDIO source is ΔΣ encoded 1-bit output from the FPGA (3.3V at 64 MHz). The 1u capacitor and 12k resistor adjusts this to line-level audio, which is +/- 0.5V AC for consumer electronics. (Note that the amplifiers and powered speakers typically provide a 10k resistor to ground to form a voltage divider.)"
Changed lines of the file:
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@@
 		(date "2023-10-01")
 		(rev "A")
+		(comment 1 "Unspecified resistors are 1% and rated for 62.5mW or higher")
+		(comment 2 "Unspecified capacitors are rated for 25V or higher")
+		(comment 3 "Signals with B-prefix are level-shifted from 3V3 to 5V")
 	)
 	(junction
@@
 			(width 0)
 			(type default)
+		)
+	)
+	(text "Audio"
+		(exclude_from_sim no)
+		(at 34.29 57.15 0)
+		(effects
+			(font
+				(size 1.5 1.5)
+				(thickness 0.8)
+				(bold yes)
+			)
+			(justify left bottom)
 		)
 	)
@@
 		)
 	)
-	(text "The AUDIO source is ΔΣ encoded 1-bit\noutput from the FPGA (3.3V at 64 MHz).\n\nThe 1u capacitor and 12k resistor\nadjusts this to line-level audio, which\nis +/- 0.5V AC for consumer electronics.\n\n(Note that the amplifiers and powered\nspeakers typically provide a 10k resistor\nto ground to form a voltage divider.)"
+	(text "PET CB2 and DIAG are inputs to FPGA.\nFPGA implements AND gate and outputs\nAUDIO source.  This saves an IC and\nallows for experimental enhancements,\nlike SID emulation at $8F00.\n\nThe AUDIO source is ΔΣ encoded 1-bit\noutput from the FPGA (3V3 at 64 MHz).\n\nThe 1u capacitor and 12k resistor\nadjusts this to line-level audio, which\nis +/- 0.5V AC for consumer electronics.\n\n(Note that amplifiers and powered speakers\ntypically provide a 10k resistor to ground\nto form a voltage divider.)"
 		(exclude_from_sim no)
-		(at 34.544 78.994 0)
+		(at 34.29 74.93 0)
 		(effects
 			(font

Commit message: hw: tidy schematics for publication
Other:
- company: (none) -> https://is.gd/6hpvh6
Changed lines of the file:
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@@
 		(date "2023-10-01")
 		(rev "A")
-		(comment 1 "Unspecified resistors are 1% and rated for 62.5mW or higher")
-		(comment 2 "Unspecified capacitors are rated for 25V or higher")
+		(company "https://is.gd/6hpvh6")
+		(comment 1 "Unspecified resistors are 1% / 62.5mW")
+		(comment 2 "Unspecified capacitors are 25V")
 		(comment 3 "Signals with B-prefix are level-shifted from 3V3 to 5V")
+		(comment 4 "License: CC0 1.0 Universal (Public Domain Dedication)")
 	)
 	(junction
