File: hw/rev-a/mainboard/kicad/IEEE.kicad_sch (KiCad schematic)
At the start: 26 parts, among them J1 IEEE, J14 IEEE_HEADER, U14 SN74LS07, U15 SN74LS07, U16 SN74LS07, U17 74LS245, U18 74LS245

Commit message: hw: ren rev-c -> rev-a
Parts:
- C75: renamed from C74; value 4.7u 10V -> 4u7 10V
- J1: footprint Retrocomputing:CBM_PET_IEEE_EDGE_CON_24P -> EconoPET:CBM_PET_IEEE_EDGE_CON_24P; symbol Retrocomputing:CBM_PET_IEEE_Conn_02x12_Card_Edge -> EconoPET:CBM_PET_IEEE_Conn_02x12_Card_Edge
- RN1: renamed from RN5; value 10k -> 10kx4
- RN11, RN12, RN13: value 470 -> 470x4
- RN2: renamed from RN1; value 4k7 -> 4k7x4
- RN3: renamed from RN2; value 4k7 -> 4k7x4
- RN4: renamed from RN6; value 10k -> 10kx4
- RN5: renamed from RN7; value 10k -> 10kx4
- RN6: renamed from RN4; value 4k7 -> 4k7x4
- RN7: renamed from RN3; value 4k7 -> 4k7x4
- RN8: value 10k -> 10kx4
- U14, U15, U16: symbol Mainboard-rescue:SN74LS07-PET -> EconoPET:SN74LS07
- renumbered C69 to C70, C70 to C71, C71 to C72, C72 to C73, C73 to C74, J14 to J20, R23 to R30, R24 to R31
Connections:
- net PD_GND is gone; now on net GND: C75.2, J1.E (GND), J1.F (GND), J1.H (GND), J1.J (GND), J1.K (GND), J1.L (GND), J1.M (GND), J1.N (GND), J20.1 (Pin_1), J20.2 (Pin_2)
Other:
- note added: "This is an approximation of the MC3446 transciever using commonly available parts. The MC3446 internally used a 2.4k/5k voltage divider. We substitute 4.7k/10k because the selection of resistor network arrays is limited from our mfgr (unless we pay a loading fee.) '07 drivers can sink 40ma, which is close to IEEE standard of 48ma. '245 recievers provide: • TTL → CMOS level conversion • Hysterises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"
- note removed: "This is an approximation of the MC3446 transciever using commonly available parts. The MC3446 internally used a 2.4k/5k voltage divider. We substitute the more common values of 4.7k/10k. '07 drivers can sink 40ma, which is close to IEEE standard of 48ma. '245 recievers provide: • TTL → CMOS level conversion • Hysterises • Hi-Z inputs to avoid loading driver 470 ohm resistors protect PIAs and VIA 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"

Commit message: hw: tidy schematics for publication
Parts:
- J1: value IEEE -> IEEE_EDGE
Other:
- note added: "IEEE-488"
- moved on the sheet: C75, J20
Changed lines of the file:
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@@
 		(date "2023-10-01")
 		(rev "A")
+		(comment 1 "Unspecified resistors are 1% and rated for 62.5mW or higher")
+		(comment 2 "Unspecified capacitors are rated for 25V or higher")
+		(comment 3 "Signals with B-prefix are level-shifted from 3V3 to 5V")
 	)
 	(bus_alias "IEEE"
@@
 	)
 	(junction
-		(at 228.6 41.91)
+		(at 231.14 48.26)
 		(diameter 0)
 		(color 0 0 0 0)
@@
 	)
 	(junction
-		(at 212.09 49.53)
+		(at 214.63 55.88)
 		(diameter 0)
 		(color 0 0 0 0)
@@
 	)
 	(junction
-		(at 219.71 49.53)
+		(at 222.25 55.88)
 		(diameter 0)
 		(color 0 0 0 0)
@@
 	(wire
 		(pts
-			(xy 228.6 41.91) (xy 228.6 43.18)
+			(xy 231.14 48.26) (xy 231.14 49.53)
 		)
 		(stroke
@@
 	(wire
 		(pts
-			(xy 204.47 44.45) (xy 205.74 44.45)
+			(xy 207.01 50.8) (xy 208.28 50.8)
 		)
 		(stroke
@@
 	(wire
 		(pts
-			(xy 212.09 49.53) (xy 219.71 49.53)
+			(xy 214.63 55.88) (xy 222.25 55.88)
 		)
 		(stroke
@@
 	(wire
 		(pts
-			(xy 204.47 49.53) (xy 204.47 44.45)
+			(xy 207.01 55.88) (xy 207.01 50.8)
 		)
 		(stroke
@@
 	(wire
 		(pts
-			(xy 228.6 48.26) (xy 228.6 49.53)
+			(xy 231.14 54.61) (xy 231.14 55.88)
 		)
 		(stroke
@@
 	(wire
 		(pts
-			(xy 218.44 44.45) (xy 219.71 44.45)
+			(xy 220.98 50.8) (xy 222.25 50.8)
 		)
 		(stroke
@@
 	(wire
 		(pts
-			(xy 218.44 41.91) (xy 228.6 41.91)
+			(xy 220.98 48.26) (xy 231.14 48.26)
 		)
 		(stroke
@@
 	(wire
 		(pts
-			(xy 212.09 49.53) (xy 204.47 49.53)
+			(xy 214.63 55.88) (xy 207.01 55.88)
 		)
 		(stroke
@@
 	(wire
 		(pts
-			(xy 219.71 44.45) (xy 219.71 49.53)
+			(xy 222.25 50.8) (xy 222.25 55.88)
 		)
 		(stroke
@@
 	(wire
 		(pts
-			(xy 219.71 49.53) (xy 228.6 49.53)
+			(xy 222.25 55.88) (xy 231.14 55.88)
 		)
 		(stroke
@@
 		)
 	)
-	(text "This is an approximation of the MC3446 transciever\nusing commonly available parts.\n\nThe MC3446 internally used a 2.4k/5k voltage divider.\nWe substitute 4.7k/10k because the selection of resistor\nnetwork arrays is limited from our mfgr (unless we pay\na loading fee.)\n\n'07 drivers can sink 40ma, which is close to IEEE\nstandard of 48ma.\n\n'245 recievers provide:\n• TTL → CMOS level conversion\n• Hysterises\n• Hi-Z inputs to avoid loading driver\n\n470Ω resistors reduce stress on the PIAs and VIA in\ncase *_IN are accidentally configured as outputs."
+	(text "This is an approximation of the MC3446 transciever\nusing commonly available parts.\n\nThe MC3446 internally used a 2.4k/5k voltage divider.\nWe substitute 4.7k/10k because the selection of resistor\nnetwork arrays is limited from our mfgr (unless we pay\na loading fee.)\n\n'07 drivers can sink 40ma, which is close to IEEE\nstandard of 48ma.\n\n'245 recievers provide:\n• TTL → CMOS level conversion\n• Hysterises\n• Hi-Z inputs to avoid loading driver\n\n470Ω resistors protect the PIAs and VIA in case\n*_IN are accidentally configured as outputs."
 		(exclude_from_sim no)
 		(at 95.25 127 0)
@@
 		)
 	)
+	(text "IEEE-488"
+		(exclude_from_sim no)
+		(at 95.25 88.9 0)
+		(effects
+			(font
+				(size 1.5 1.5)
+				(thickness 0.8)
+				(bold yes)
+			)
+			(justify left bottom)
+		)
+	)
 	(label "DIO7"
-		(at 218.44 29.21 0)
+		(at 220.98 35.56 0)
 		(fields_autoplaced yes)
 		(effects
@@
 	)
 	(label "ATN"
-		(at 205.74 41.91 180)
+		(at 208.28 48.26 180)
 		(fields_autoplaced yes)
 		(effects
@@
 	)
 	(label "DIO6"
-		(at 218.44 26.67 0)
+		(at 220.98 33.02 0)
 		(fields_autoplaced yes)
 		(effects
@@
 	)
 	(label "IFC"
-		(at 205.74 39.37 180)
+		(at 208.28 45.72 180)
 		(fields_autoplaced yes)
 		(effects
@@
 	)
 	(label "DIO1"
-		(at 205.74 24.13 180)
+		(at 208.28 30.48 180)
 		(fields_autoplaced yes)
 		(effects
@@
 	)
 	(label "SRQ"
-		(at 218.44 39.37 0)
+		(at 220.98 45.72 0)
 		(fields_autoplaced yes)
 		(effects
@@
 	)
 	(label "DIO4"
-		(at 205.74 31.75 180)
+		(at 208.28 38.1 180)
 		(fields_autoplaced yes)
 		(effects
@@
 	)
 	(label "EOI"
-		(at 205.74 34.29 180)
+		(at 208.28 40.64 180)
 		(fields_autoplaced yes)
 		(effects
@@
 	)
 	(label "DIO3"
-		(at 205.74 29.21 180)
+		(at 208.28 35.56 180)
 		(fields_autoplaced yes)
 		(effects
@@
 	)
 	(label "DAV"
-		(at 218.44 34.29 0)
+		(at 220.98 40.64 0)
 		(fields_autoplaced yes)
 		(effects
@@
 	)
 	(label "DIO5"
-		(at 218.44 24.13 0)
+		(at 220.98 30.48 0)
 		(fields_autoplaced yes)
 		(effects
@@
 	)
 	(label "NDAC"
-		(at 218.44 36.83 0)
+		(at 220.98 43.18 0)
 		(fields_autoplaced yes)
 		(effects
@@
 	)
 	(label "DIO8"
-		(at 218.44 31.75 0)
+		(at 220.98 38.1 0)
 		(fields_autoplaced yes)
 		(effects
@@
 	)
 	(label "NRFD"
-		(at 205.74 36.83 180)
+		(at 208.28 43.18 180)
 		(fields_autoplaced yes)
 		(effects
@@
 	)
 	(label "DIO2"
-		(at 205.74 26.67 180)
+		(at 208.28 33.02 180)
 		(fields_autoplaced yes)
 		(effects
@@
 			)
 		)
-		(property "Value" "IEEE"
+		(property "Value" "IEEE_EDGE"
 			(at 240.03 103.4796 0)
 			(effects
@@
 	(symbol
 		(lib_id "Connector_Generic:Conn_02x09_Odd_Even")
-		(at 210.82 34.29 0)
+		(at 213.36 40.64 0)
 		(mirror x)
 		(unit 1)
@@
 		(fields_autoplaced yes)
 		(property "Reference" "J20"
-			(at 212.09 17.78 0)
+			(at 214.63 24.13 0)
 			(effects
 				(font
@@
 		)
 		(property "Value" "IEEE_HEADER"
-			(at 212.09 20.32 0)
+			(at 214.63 26.67 0)
 			(effects
 				(font
@@
 		)
 		(property "Footprint" "Connector_PinHeader_2.54mm:PinHeader_2x09_P2.54mm_Vertical"
-			(at 210.82 34.29 0)
+			(at 213.36 40.64 0)
 			(effects
 				(font
@@
 		)
 		(property "Datasheet" "~"
-			(at 210.82 34.29 0)
+			(at 213.36 40.64 0)
 			(effects
 				(font
@@
 		)
 		(property "Description" ""
-			(at 210.82 34.29 0)
+			(at 213.36 40.64 0)
 			(effects
 				(font
@@
 		)
 		(property "MOUSER" "649-1012938195002BLF"
-			(at 210.82 34.29 0)
+			(at 213.36 40.64 0)
 			(effects
 				(font
@@
 	(symbol
 		(lib_id "Device:C_Small")
-		(at 228.6 45.72 0)
+		(at 231.14 52.07 0)
 		(unit 1)
 		(exclude_from_sim no)
@@
 		(dnp no)
 		(property "Reference" "C75"
-			(at 230.9368 44.5516 0)
+			(at 233.4768 50.9016 0)
 			(effects
 				(font
@@
 		)
 		(property "Value" "4u7 10V"
-			(at 230.9368 46.863 0)
+			(at 233.4768 53.213 0)
 			(effects
 				(font
@@
 		)
 		(property "Footprint" "Capacitor_SMD:C_0402_1005Metric"
-			(at 228.6 45.72 0)
+			(at 231.14 52.07 0)
 			(effects
 				(font
@@
 		)
 		(property "Datasheet" "https://product.samsungsem.com/mlcc/CL05A475MP5NRN.do"
-			(at 228.6 45.72 0)
+			(at 231.14 52.07 0)
 			(effects
 				(font
@@
 		)
 		(property "Description" ""
-			(at 228.6 45.72 0)
+			(at 231.14 52.07 0)
 			(effects
 				(font
@@
 		)
 		(property "LCSC" "C23733"
-			(at 228.6 45.72 0)
+			(at 231.14 52.07 0)
 			(effects
 				(font
@@
 	(symbol
 		(lib_id "power:GND")
-		(at 212.09 49.53 0)
+		(at 214.63 55.88 0)
 		(unit 1)
 		(exclude_from_sim no)
@@
 		(fields_autoplaced yes)
 		(property "Reference" "#PWR0113"
-			(at 212.09 55.88 0)
+			(at 214.63 62.23 0)
 			(effects
 				(font
@@
 		)
 		(property "Value" "GND"
-			(at 212.09 54.61 0)
+			(at 214.63 60.96 0)
 			(effects
 				(font
@@
 		)
 		(property "Footprint" ""
-			(at 212.09 49.53 0)
+			(at 214.63 55.88 0)
 			(effects
 				(font
@@
 		)
 		(property "Datasheet" ""
-			(at 212.09 49.53 0)
+			(at 214.63 55.88 0)
 			(effects
 				(font
@@
 		)
 		(property "Description" "Power symbol creates a global label with name \"GND\" , ground"
-			(at 212.09 49.53 0)
+			(at 214.63 55.88 0)
 			(effects
 				(font
@@
 	(symbol
 		(lib_id "power:+5V")
-		(at 228.6 41.91 0)
+		(at 231.14 48.26 0)
 		(unit 1)
 		(exclude_from_sim no)
@@
 		(fields_autoplaced yes)
 		(property "Reference" "#PWR0114"
-			(at 228.6 45.72 0)
+			(at 231.14 52.07 0)
 			(effects
 				(font
@@
 		)
 		(property "Value" "+5V"
-			(at 228.6 36.83 0)
+			(at 231.14 43.18 0)
 			(effects
 				(font
@@
 		)
 		(property "Footprint" ""
-			(at 228.6 41.91 0)
+			(at 231.14 48.26 0)
 			(effects
 				(font
@@
 		)
 		(property "Datasheet" ""
-			(at 228.6 41.91 0)
+			(at 231.14 48.26 0)
 			(effects
 				(font
@@
 		)
 		(property "Description" "Power symbol creates a global label with name \"+5V\""
-			(at 228.6 41.91 0)
+			(at 231.14 48.26 0)
 			(effects
 				(font

Commit message: hw: tidy schematics for publication
Other:
- company: (none) -> https://is.gd/6hpvh6
Changed lines of the file:
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@@
 		(date "2023-10-01")
 		(rev "A")
-		(comment 1 "Unspecified resistors are 1% and rated for 62.5mW or higher")
-		(comment 2 "Unspecified capacitors are rated for 25V or higher")
+		(company "https://is.gd/6hpvh6")
+		(comment 1 "Unspecified resistors are 1% / 62.5mW")
+		(comment 2 "Unspecified capacitors are 25V")
 		(comment 3 "Signals with B-prefix are level-shifted from 3V3 to 5V")
+		(comment 4 "License: CC0 1.0 Universal (Public Domain Dedication)")
 	)
 	(bus_alias "IEEE"
