File: hw/rev-a/mainboard/kicad/Mainboard.kicad_sch (KiCad schematic)
At the start: 0 parts

Commit message: hw: tidy schematics for publication
Other:
- note added: ""If you don't use a current limiting resistor the LED will light up orange! Because of the fire! Because sometimes Daddy makes mistakes." - Milo, Age 4.5"
- note added: "System Block Diagram"
- company: (none) -> https://is.gd/6hpvh6
Changed lines of the file:
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@@
 		(date "2023-10-01")
 		(rev "A")
+		(company "https://is.gd/6hpvh6")
+		(comment 1 "Unspecified resistors are 1% and rated for 62.5mW or higher")
+		(comment 2 "Unspecified capacitors are rated for 25V or higher")
+		(comment 3 "Signals with B-prefix are level-shifted from 3V3 to 5V")
+		(comment 4 "License: CC0 1.0 Universal (Public Domain Dedication)")
 	)
 	(junction
@@
 	)
 	(junction
-		(at 209.55 100.33)
-		(diameter 0)
-		(color 0 0 0 0)
-	)
-	(junction
 		(at 109.22 134.62)
 		(diameter 0)
@@
 	)
 	(junction
-		(at 212.09 102.87)
+		(at 163.83 129.54)
 		(diameter 0)
 		(color 0 0 0 0)
 	)
 	(junction
-		(at 163.83 129.54)
+		(at 205.74 105.41)
 		(diameter 0)
 		(color 0 0 0 0)
@@
 	)
 	(junction
-		(at 214.63 105.41)
+		(at 200.66 100.33)
 		(diameter 0)
 		(color 0 0 0 0)
@@
 	)
 	(junction
+		(at 203.2 102.87)
+		(diameter 0)
+		(color 0 0 0 0)
+	)
+	(junction
 		(at 149.86 93.98)
 		(diameter 0)
@@
 	(wire
 		(pts
-			(xy 152.4 180.34) (xy 60.96 180.34)
-		)
-		(stroke
-			(width 0)
-			(type default)
-		)
-	)
-	(wire
-		(pts
-			(xy 149.86 177.8) (xy 63.5 177.8)
+			(xy 152.4 176.53) (xy 60.96 176.53)
+		)
+		(stroke
+			(width 0)
+			(type default)
+		)
+	)
+	(wire
+		(pts
+			(xy 149.86 173.99) (xy 63.5 173.99)
 		)
 		(stroke
@@
 	(wire
 		(pts
+			(xy 203.2 102.87) (xy 212.09 102.87)
+		)
+		(stroke
+			(width 0)
+			(type default)
+		)
+	)
+	(wire
+		(pts
 			(xy 142.24 41.91) (xy 168.91 41.91)
 		)
@@
 	(wire
 		(pts
-			(xy 194.31 100.33) (xy 209.55 100.33)
+			(xy 194.31 100.33) (xy 200.66 100.33)
 		)
 		(stroke
@@
 	(wire
 		(pts
-			(xy 147.32 90.17) (xy 147.32 175.26)
+			(xy 147.32 90.17) (xy 147.32 171.45)
 		)
 		(stroke
@@
 	(wire
 		(pts
-			(xy 214.63 105.41) (xy 214.63 166.37)
+			(xy 205.74 105.41) (xy 205.74 166.37)
 		)
 		(stroke
@@
 	(wire
 		(pts
-			(xy 194.31 105.41) (xy 214.63 105.41)
+			(xy 194.31 105.41) (xy 205.74 105.41)
 		)
 		(stroke
@@
 	(wire
 		(pts
-			(xy 66.04 175.26) (xy 66.04 134.62)
+			(xy 66.04 171.45) (xy 66.04 134.62)
 		)
 		(stroke
@@
 	(wire
 		(pts
-			(xy 209.55 100.33) (xy 220.98 100.33)
-		)
-		(stroke
-			(width 0)
-			(type default)
-		)
-	)
-	(wire
-		(pts
 			(xy 163.83 105.41) (xy 163.83 129.54)
 		)
@@
 	(wire
 		(pts
-			(xy 194.31 102.87) (xy 212.09 102.87)
+			(xy 194.31 102.87) (xy 203.2 102.87)
+		)
+		(stroke
+			(width 0)
+			(type default)
+		)
+	)
+	(wire
+		(pts
+			(xy 200.66 100.33) (xy 212.09 100.33)
 		)
 		(stroke
@@
 	(wire
 		(pts
-			(xy 63.5 177.8) (xy 63.5 132.08)
+			(xy 63.5 173.99) (xy 63.5 132.08)
 		)
 		(stroke
@@
 	(wire
 		(pts
-			(xy 212.09 102.87) (xy 220.98 102.87)
-		)
-		(stroke
-			(width 0)
-			(type default)
-		)
-	)
-	(wire
-		(pts
 			(xy 114.3 31.75) (xy 116.84 31.75)
 		)
@@
 	(wire
 		(pts
-			(xy 60.96 180.34) (xy 60.96 129.54)
+			(xy 60.96 176.53) (xy 60.96 129.54)
 		)
 		(stroke
@@
 	(wire
 		(pts
-			(xy 147.32 175.26) (xy 66.04 175.26)
+			(xy 147.32 171.45) (xy 66.04 171.45)
 		)
 		(stroke
@@
 	(wire
 		(pts
-			(xy 214.63 105.41) (xy 220.98 105.41)
-		)
-		(stroke
-			(width 0)
-			(type default)
-		)
-	)
-	(wire
-		(pts
 			(xy 168.91 96.52) (xy 152.4 96.52)
 		)
@@
 	(wire
 		(pts
+			(xy 205.74 105.41) (xy 212.09 105.41)
+		)
+		(stroke
+			(width 0)
+			(type default)
+		)
+	)
+	(wire
+		(pts
 			(xy 114.3 24.13) (xy 148.59 24.13)
 		)
@@
 	(wire
 		(pts
-			(xy 209.55 161.29) (xy 114.3 161.29)
+			(xy 200.66 161.29) (xy 114.3 161.29)
 		)
 		(stroke
@@
 	(wire
 		(pts
-			(xy 209.55 100.33) (xy 209.55 161.29)
+			(xy 200.66 100.33) (xy 200.66 161.29)
 		)
 		(stroke
@@
 	(wire
 		(pts
-			(xy 212.09 102.87) (xy 212.09 163.83)
+			(xy 203.2 102.87) (xy 203.2 163.83)
 		)
 		(stroke
@@
 	(wire
 		(pts
-			(xy 212.09 163.83) (xy 111.76 163.83)
+			(xy 203.2 163.83) (xy 111.76 163.83)
 		)
 		(stroke
@@
 	(wire
 		(pts
-			(xy 152.4 96.52) (xy 152.4 180.34)
+			(xy 152.4 96.52) (xy 152.4 176.53)
 		)
 		(stroke
@@
 	(wire
 		(pts
-			(xy 214.63 166.37) (xy 109.22 166.37)
+			(xy 205.74 166.37) (xy 109.22 166.37)
 		)
 		(stroke
@@
 	(wire
 		(pts
-			(xy 149.86 93.98) (xy 149.86 177.8)
+			(xy 149.86 93.98) (xy 149.86 173.99)
 		)
 		(stroke
@@
 			(width 0)
 			(type default)
+		)
+	)
+	(text "\"If you don't use a current limiting resistor the\n LED will light up orange!  Because of the fire!\n Because sometimes Daddy makes mistakes.\"\n\n                                - Milo, Age 4.5\n"
+		(exclude_from_sim no)
+		(at 76.2 190.5 0)
+		(effects
+			(font
+				(size 1.5875 1.5875)
+				(thickness 0.3175)
+				(bold yes)
+				(italic yes)
+			)
+			(justify left)
+		)
+	)
+	(text "System Block Diagram"
+		(exclude_from_sim no)
+		(at 40.64 20.32 0)
+		(effects
+			(font
+				(size 1.5 1.5)
+				(thickness 0.8)
+				(bold yes)
+			)
+			(justify left bottom)
 		)
 	)
@@
 	)
 	(sheet
-		(at 220.98 29.21)
+		(at 212.09 73.66)
 		(size 20.32 11.43)
 		(fields_autoplaced yes)
@@
 		)
 		(property "Sheetname" "POWER"
-			(at 220.98 28.4984 0)
+			(at 212.09 72.9484 0)
 			(effects
 				(font
@@
 		)
 		(property "Sheetfile" "POWER.kicad_sch"
-			(at 220.98 41.2246 0)
+			(at 212.09 85.6746 0)
 			(effects
 				(font
@@
 	)
 	(sheet
-		(at 220.98 97.79)
+		(at 212.09 97.79)
 		(size 20.32 11.43)
 		(fields_autoplaced yes)
@@
 		)
 		(property "Sheetname" "VIDEO"
-			(at 220.98 97.0784 0)
+			(at 212.09 97.0784 0)
 			(effects
 				(font
@@
 		)
 		(property "Sheetfile" "VIDEO.kicad_sch"
-			(at 220.98 109.8046 0)
+			(at 212.09 109.8046 0)
 			(effects
 				(font
@@
 		)
 		(pin "BVERT" input
-			(at 220.98 105.41 180)
+			(at 212.09 105.41 180)
 			(effects
 				(font
@@
 		)
 		(pin "BVIDEO" input
-			(at 220.98 100.33 180)
+			(at 212.09 100.33 180)
 			(effects
 				(font
@@
 		)
 		(pin "BHORIZ" input
-			(at 220.98 102.87 180)
-			(effects
-				(font
+			(at 212.09 102.87 180)
+			(effects
+				(font
