File: hw/rev-a/mainboard/kicad/MicroSD.kicad_sch (KiCad schematic)
At the start: 5 parts, among them J25 MICRO_SD

Commit message: hw: tidy schematics for publication
Other:
- note added: "47uF decoupling capacitor helps inrush current (although hot insertion is not recommended)."
- note added: "DAT[0] : (POCI) is open-drain output that requires pullup. DAT[2:1] : Unused inputs in SPI mode. Pullups recommended to avoid current draw due to metastablitiy. DAT[3] : (~{CS}) has built-in 22-50k pullup to ensure card is deselected by default. CMD : (PICO) input in SPI mode. CLK : (SCK) always an input. Never gets pullup. For reference, CM1624 uses: 25k pullup for DAT[0:3] and CMD 40 Ohm termin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"
- note removed: "47uF decoupling capacitor handles inrush current from hot insertion."
- note removed: "DAT[0] : (POCI) is open-drain output that requires pullup. DAT[2:1] : Unused inputs in SPI mode. Pullups recommended to avoid current draw due to metastablitiy. DAT[3] : (~{CS}) has built-in 22-50k pullup to ensure card is deselected by default. CMD : (PICO) input in SPI mode. CLK : (SCK) always an input. Never gets pullup. CM1624 uses: 25k pullup for DAT[0:3] and CMD 40 Ohm termination for DAT[0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"
Changed lines of the file:
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@@
 		(date "2023-10-01")
 		(rev "A")
+		(comment 1 "Unspecified resistors are 1% and rated for 62.5mW or higher")
+		(comment 2 "Unspecified capacitors are rated for 25V or higher")
+		(comment 3 "Signals with B-prefix are level-shifted from 3V3 to 5V")
 	)
 	(junction
@@
 		)
 	)
-	(text "47uF decoupling capacitor handles\ninrush current from hot insertion."
+	(text "47uF decoupling capacitor helps inrush current\n(although hot insertion is not recommended)."
 		(exclude_from_sim no)
-		(at 180.34 71.12 0)
+		(at 179.07 72.39 0)
 		(effects
 			(font
@@
 		)
 	)
-	(text "DAT[0]   : (POCI) is open-drain output that requires pullup.\nDAT[2:1] : Unused inputs in SPI mode.  Pullups recommended\n           to avoid current draw due to metastablitiy.\nDAT[3]   : (~{CS}) has built-in 22-50k pullup to ensure card\n           is deselected by default.\nCMD      : (PICO) input in SPI mode.\nCLK      : (SCK) always an input.  Never gets pullup.\n\nCM1624 uses:\n25k pullup for DAT[0:3] and CMD\n40 Ohm termination for DAT[0:3], CMD, and CLK\n\n10k pullups common (e.g., ExpressIf documentation)."
+	(text "DAT[0]   : (POCI) is open-drain output that requires pullup.\nDAT[2:1] : Unused inputs in SPI mode.  Pullups recommended\n           to avoid current draw due to metastablitiy.\nDAT[3]   : (~{CS}) has built-in 22-50k pullup to ensure card\n           is deselected by default.\nCMD      : (PICO) input in SPI mode.\nCLK      : (SCK) always an input.  Never gets pullup.\n\nFor reference, CM1624 uses:\n25k pullup for DAT[0:3] and CMD\n40 Ohm termination for DAT[0:3], CMD, and CLK\n\n10k pullups common (e.g., ExpressIf documentation)."
 		(exclude_from_sim no)
-		(at 153.67 149.86 0)
+		(at 153.67 153.67 0)
 		(effects
 			(font
@@
 	(text "MicroSD"
 		(exclude_from_sim no)
-		(at 100.33 63.5 0)
+		(at 153.67 125.73 0)
 		(effects
 			(font

Commit message: hw: tidy schematics for publication
Other:
- company: (none) -> https://is.gd/6hpvh6
Changed lines of the file:
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@@
 		(date "2023-10-01")
 		(rev "A")
-		(comment 1 "Unspecified resistors are 1% and rated for 62.5mW or higher")
-		(comment 2 "Unspecified capacitors are rated for 25V or higher")
+		(company "https://is.gd/6hpvh6")
+		(comment 1 "Unspecified resistors are 1% / 62.5mW")
+		(comment 2 "Unspecified capacitors are 25V")
 		(comment 3 "Signals with B-prefix are level-shifted from 3V3 to 5V")
+		(comment 4 "License: CC0 1.0 Universal (Public Domain Dedication)")
 	)
 	(junction
