File: hw/rev-a/mainboard/kicad/USB.kicad_sch (KiCad schematic)
At the start: 6 parts, among them J26 USB1.1_HOST_TYPE_C

Commit message: hw: tidy schematics for publication
Other:
- note added: "USB"
- note added: "USB 1.1 Host over USB-C connector The 56k pullups on CC1 and CC2 identify the port as downstream facing, supplying 5V/900ma. The diode prevents connected devices from inadvertently backpowering the EconoPET. V_{F} < 0.5V should be within USB spec of 5V +/-10%. The 47u capacitor helps with current inrush (although hot insertion is not recommened.) Consider using an independently powered USB hub as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"
- note removed: "USB 1.1 Host over USB-C connector The 56k pullups on CC1 and CC2 identify the port as downstream facing, supplying 5V/900ma. The diode prevents connected devices from inadvertently backpowering the EconoPET. V_{F} < 0.5V should be within USB spec of 5V +/-10%. An independently powered USB hub is recommended as an extra layer of protection against devices that incorrectly draw excessive current."
- moved on the sheet: C102, C103, D12, J26, R63, R64

Commit message: hw: tidy schematics for publication
Other:
- company: (none) -> https://is.gd/6hpvh6
Changed lines of the file:
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@@
 		(date "2023-10-01")
 		(rev "A")
-		(comment 1 "Unspecified resistors are 1% and rated for 62.5mW or higher")
-		(comment 2 "Unspecified capacitors are rated for 25V or higher")
+		(company "https://is.gd/6hpvh6")
+		(comment 1 "Unspecified resistors are 1% / 62.5mW")
+		(comment 2 "Unspecified capacitors are 25V")
 		(comment 3 "Signals with B-prefix are level-shifted from 3V3 to 5V")
+		(comment 4 "License: CC0 1.0 Universal (Public Domain Dedication)")
 	)
 	(junction
