File: hw/rev-a/mainboard/kicad/VIDEO.kicad_sch (KiCad schematic)
At the start: 1 part, among them J7 VIDEO

Commit message: hw: tidy schematics for publication
Other:
- note added: "VIDEO HEADER"
Changed lines of the file:
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@@
 		(date "2023-10-01")
 		(rev "A")
+		(comment 1 "Unspecified resistors are 1% and rated for 62.5mW or higher")
+		(comment 2 "Unspecified capacitors are rated for 25V or higher")
+		(comment 3 "Signals with B-prefix are level-shifted from 3V3 to 5V")
 	)
 	(junction
@@
 		)
 	)
+	(text "VIDEO HEADER"
+		(exclude_from_sim no)
+		(at 124.46 80.01 0)
+		(effects
+			(font
+				(size 1.5 1.5)
+				(thickness 0.8)
+				(bold yes)
+			)
+			(justify left bottom)
+		)
+	)

Commit message: hw: tidy schematics for publication
Other:
- note added: "Not too much to see here. :-) If you're looking for the modern DVI video output over an HDMI connector, look under Magic / MCU / DVI."
- company: (none) -> https://is.gd/6hpvh6
Changed lines of the file:
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@@
 		(date "2023-10-01")
 		(rev "A")
-		(comment 1 "Unspecified resistors are 1% and rated for 62.5mW or higher")
-		(comment 2 "Unspecified capacitors are rated for 25V or higher")
+		(company "https://is.gd/6hpvh6")
+		(comment 1 "Unspecified resistors are 1% / 62.5mW")
+		(comment 2 "Unspecified capacitors are 25V")
 		(comment 3 "Signals with B-prefix are level-shifted from 3V3 to 5V")
+		(comment 4 "License: CC0 1.0 Universal (Public Domain Dedication)")
 	)
 	(junction
@@
 		)
 	)
+	(text "Not too much to see here.  :-)\n\nIf you're looking for the modern DVI\nvideo output over an HDMI connector,\nlook under Magic / MCU / DVI."
+		(exclude_from_sim no)
+		(at 123.19 115.57 0)
+		(effects
+			(font
+				(size 1.27 1.27)
+			)
+			(justify left)
+		)
+	)
