File: hw/rev-a/mainboard/kicad/DVI.kicad_sch (KiCad schematic)
At the start: 14 parts, among them J24 NOT_HDMI_A

Commit message: hw: tidy schematics for publication
Other:
- note added: "CEC, SCL, and SDA are for experimentation and disconnected by solder jumpers by default. DANGER: Closing the DVI_SCL/DVI_SDA jumpers pulls the corresponding RP2040 GPIO pins to +5V. Only do this if you know what you're doing."
- note added: "Uses legacy DVI TMDS protocol over an HDMI connector. See: https://github.com/Wren6991/PicoDVI"
- note removed: "CEC, SCL, and SDA are for possible future use and disconnected by solder jumpers by default. DANGER: Closing the DVI_SCL/DVI_SDA jumpers pulls the corresponding RP2040 GPIO pins to +5V. Only do this if you know what you're doing."
- note removed: "Technically, not true HDMI. This is the DVI TMDS protocol over an HDMI connector."
- company: (none) -> https://is.gd/6hpvh6
Changed lines of the file:
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@@
 		(date "2023-10-01")
 		(rev "A")
-		(comment 1 "Unspecified resistors are 1% and rated for 62.5mW or higher")
-		(comment 2 "Unspecified capacitors are rated for 25V or higher")
+		(company "https://is.gd/6hpvh6")
+		(comment 1 "Unspecified resistors are 1% / 62.5mW")
+		(comment 2 "Unspecified capacitors are 25V")
 		(comment 3 "Signals with B-prefix are level-shifted from 3V3 to 5V")
+		(comment 4 "License: CC0 1.0 Universal (Public Domain Dedication)")
 	)
 	(bus_alias "DVI"
@@
 		)
 	)
-	(text "CEC, SCL, and SDA are for possible future use and\ndisconnected by solder jumpers by default.\n\nDANGER: Closing the DVI_SCL/DVI_SDA jumpers pulls\nthe corresponding RP2040 GPIO pins to +5V.\n\nOnly do this if you know what you're doing."
+	(text "CEC, SCL, and SDA are for experimentation and\ndisconnected by solder jumpers by default.\n\nDANGER: Closing the DVI_SCL/DVI_SDA jumpers pulls\nthe corresponding RP2040 GPIO pins to +5V.\n\nOnly do this if you know what you're doing."
 		(exclude_from_sim no)
 		(at 80.01 134.62 0)
@@
 		)
 	)
-	(text "Technically, not true HDMI.  This is the DVI\nTMDS protocol over an HDMI connector."
+	(text "Uses legacy DVI TMDS protocol over an HDMI connector.\nSee: https://github.com/Wren6991/PicoDVI"
 		(exclude_from_sim no)
-		(at 83.82 52.07 0)
+		(at 83.82 50.8 0)
 		(effects
 			(font
@@
 	(text "DVI VIDEO"
 		(exclude_from_sim no)
-		(at 83.82 48.26 0)
+		(at 83.82 45.72 0)
 		(effects
 			(font

Commit message: hw: tidy schematics for publication
Other:
- note added: "DVI TMDS protocol over an HDMI-compatible connector (not HDMI certified). See: https://github.com/Wren6991/PicoDVI"
- note removed: "Uses legacy DVI TMDS protocol over an HDMI connector. See: https://github.com/Wren6991/PicoDVI"
Changed lines of the file:
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@@
 		)
 	)
-	(text "Uses legacy DVI TMDS protocol over an HDMI connector.\nSee: https://github.com/Wren6991/PicoDVI"
+	(text "DVI TMDS protocol over an HDMI-compatible\nconnector (not HDMI certified).\n\nSee: https://github.com/Wren6991/PicoDVI"
 		(exclude_from_sim no)
-		(at 83.82 50.8 0)
+		(at 83.82 49.53 0)
 		(effects
 			(font
@@
 	(text "DVI VIDEO"
 		(exclude_from_sim no)
-		(at 83.82 45.72 0)
+		(at 83.82 43.18 0)
 		(effects
 			(font
