File: hw/rev-a/mainboard/kicad/CPU.kicad_sch (KiCad schematic)
At the start: 12 parts, among them SW1 RESET, SW2 NMI, U1 W65C02S, U2 AS6C1008

Commit message: hw: ren rev-c -> rev-a
Parts:
- C4: renamed from C24; footprint Capacitor_SMD:C_0603_1608Metric -> Capacitor_SMD:C_0402_1005Metric; LCSC C96446 -> (none); now not fitted
- C5: renamed from C23; footprint Capacitor_SMD:C_0603_1608Metric -> Capacitor_SMD:C_0402_1005Metric; LCSC C96446 -> (none); now not fitted
- SW1, SW2: footprint JLCPCB:SW-TH_L6.0-W3.5-P6.50 -> EconoPET:SW_PUSH_1P1T_6x3.5mm_H4.3_APEM_MJTP1243
- U1: symbol Mainboard-rescue:W65C02SxP-PET -> EconoPET:W65C02S
- U2: symbol Mainboard-rescue:AS6C1008-PET -> EconoPET:AS6C1008
- renumbered C20 to C100, C22 to C104
Connections:
- net PD_GND is gone; now on net GND: SW1.1, SW2.1, U1.21 (VSS), U2.16 (VSS), U2.22 (CE#)
Other:
- note added: "A single 128KB SRAM chip is used for the 32K main RAM, 64K expansion RAM, 2K display RAM, 2K character ROM and 26K system ROM. ROMs are initialized by the MCU on POR (via SPI -> bus bridge provided by the FPGA). A[15:0] are the address of the shared system bus, which is connected to the CPU, IO, FPGA and most RAM address pins. The exceptions are RAM_A[16:15,11:10], which are driven exclusively by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"
- note added: "The bus is shared with the FPGA. The FPGA deasserts BE (Bus Enable) to transition the CPU's Address, Data, and R~{W} buffers to high-Z while the FPGA drives the bus. CPU and RAM operate at +3V3 to interface directly with the FPGA. Level shifters are used for connections to the 5V I/O section. This split avoids needing level shifters for A[5..16]."
- note removed: "A single 128KB SRAM chip is used for main RAM, expansion RAM, display RAM and ROM. The ROM portion is initialized at POR by the MCU. A[15:0] are the address of the shared system bus, which is connected to the CPU, IO, FPGA and most RAM address pins. The exceptions are RAM_A[16:15,11:10], which are driven exclusively by the FPGA. RAM_A[11:10] is used by the FPGA to mirror display RAM when the CPU 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"
- note removed: "The bus is shared with the FPGA. The FPGA pulls BE (Bus Enable) low to put the CPU's Address, Data, and R~{W} buffers in to high-Z while the FPGA drives the bus. CPU and RAM operate at +3V3 to interface directly with the FPGA. Level shifters are used for connections to the 5V I/O section. This split avoids needing level shifters for A[5..16]."

Commit message: hw: tidy schematics for publication
Other:
- note added: "CPU and RAM operate at 3V3 so that the system bus and CPU control signals can be directly shared with the FPGA. Level shifters are used for connections to the 5V I/O section. This design avoids needing level shifters for A[5..16]. The FPGA deasserts BE (Bus Enable) to transition the CPU's Address, Data, and R~{W} buffers to high-Z when the FPGA drives the bus."
- note added: "To simplify routing, address and data lines are arbitrarily assigned to the address and data pins of the SRAM."
- note added: "~{RES}, ~{IRQ}, ~{NMI}, and RDY are open-drain and wire ORed. ~{SO} is driven high by the FPGA."
- note removed: "The bus is shared with the FPGA. The FPGA deasserts BE (Bus Enable) to transition the CPU's Address, Data, and R~{W} buffers to high-Z while the FPGA drives the bus. CPU and RAM operate at +3V3 to interface directly with the FPGA. Level shifters are used for connections to the 5V I/O section. This split avoids needing level shifters for A[5..16]."
- note removed: "To improve routing, address and data lines are arbitrarily assigned to the address and data pins of the SRAM."
- note removed: "~{RES}, ~{IRQ}, and ~{NMI} are open-drain and wire ORed. RDY is bidirectional and wire ORed. ~{SO} is pulled high by the FPGA."
Changed lines of the file:
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@@
 		(date "2023-10-01")
 		(rev "A")
+		(comment 1 "Unspecified resistors are 1% and rated for 62.5mW or higher")
+		(comment 2 "Unspecified capacitors are rated for 25V or higher")
+		(comment 3 "Signals with B-prefix are level-shifted from 3V3 to 5V")
 	)
 	(bus_alias "RAM_A"
@@
 	)
 	(bus_entry
-		(at 110.49 119.38)
+		(at 111.76 119.38)
 		(size 2.54 2.54)
 		(stroke
@@
 	)
 	(bus_entry
-		(at 110.49 124.46)
+		(at 111.76 124.46)
 		(size 2.54 2.54)
 		(stroke
@@
 	)
 	(bus_entry
-		(at 110.49 132.08)
+		(at 111.76 132.08)
 		(size 2.54 2.54)
 		(stroke
@@
 	)
 	(bus_entry
-		(at 110.49 137.16)
-		(size 2.54 2.54)
-		(stroke
-			(width 0)
-			(type default)
-		)
-	)
-	(bus_entry
-		(at 110.49 127)
+		(at 111.76 137.16)
+		(size 2.54 2.54)
+		(stroke
+			(width 0)
+			(type default)
+		)
+	)
+	(bus_entry
+		(at 111.76 127)
 		(size 2.54 2.54)
 		(stroke
@@
 	)
 	(bus_entry
-		(at 110.49 121.92)
+		(at 111.76 121.92)
 		(size 2.54 2.54)
 		(stroke
@@
 	)
 	(bus_entry
-		(at 110.49 129.54)
+		(at 111.76 129.54)
 		(size 2.54 2.54)
 		(stroke
@@
 	)
 	(bus_entry
-		(at 110.49 134.62)
+		(at 111.76 134.62)
 		(size 2.54 2.54)
 		(stroke
@@
 	(wire
 		(pts
+			(xy 107.95 132.08) (xy 111.76 132.08)
+		)
+		(stroke
+			(width 0)
+			(type default)
+		)
+	)
+	(wire
+		(pts
 			(xy 187.96 68.58) (xy 207.01 68.58)
 		)
@@
 		)
 	)
-	(wire
-		(pts
-			(xy 107.95 129.54) (xy 110.49 129.54)
-		)
-		(stroke
-			(width 0)
-			(type default)
-		)
-	)
-	(wire
-		(pts
-			(xy 107.95 127) (xy 110.49 127)
-		)
-		(stroke
-			(width 0)
-			(type default)
-		)
-	)
 	(bus
 		(pts
@@
 		)
 	)
+	(wire
+		(pts
+			(xy 107.95 124.46) (xy 111.76 124.46)
+		)
+		(stroke
+			(width 0)
+			(type default)
+		)
+	)
 	(bus
 		(pts
@@
 	(wire
 		(pts
+			(xy 107.95 129.54) (xy 111.76 129.54)
+		)
+		(stroke
+			(width 0)
+			(type default)
+		)
+	)
+	(wire
+		(pts
 			(xy 107.95 111.76) (xy 111.76 111.76)
 		)
@@
 	(wire
 		(pts
-			(xy 107.95 121.92) (xy 110.49 121.92)
-		)
-		(stroke
-			(width 0)
-			(type default)
-		)
-	)
-	(wire
-		(pts
 			(xy 187.96 67.31) (xy 187.96 68.58)
 		)
@@
 	(bus
 		(pts
-			(xy 113.03 129.54) (xy 113.03 132.08)
+			(xy 114.3 129.54) (xy 114.3 132.08)
 		)
 		(stroke
@@
 	(wire
 		(pts
-			(xy 107.95 132.08) (xy 110.49 132.08)
-		)
-		(stroke
-			(width 0)
-			(type default)
-		)
-	)
-	(wire
-		(pts
 			(xy 53.34 127) (xy 77.47 127)
 		)
@@
 		)
 	)
+	(wire
+		(pts
+			(xy 107.95 134.62) (xy 111.76 134.62)
+		)
+		(stroke
+			(width 0)
+			(type default)
+		)
+	)
 	(bus
 		(pts
@@
 	(bus
 		(pts
-			(xy 113.03 146.05) (xy 113.03 139.7)
+			(xy 114.3 142.24) (xy 114.3 139.7)
 		)
 		(stroke
@@
 	(bus
 		(pts
-			(xy 113.03 124.46) (xy 113.03 127)
+			(xy 114.3 124.46) (xy 114.3 127)
 		)
 		(stroke
@@
 	(wire
 		(pts
+			(xy 107.95 137.16) (xy 111.76 137.16)
+		)
+		(stroke
+			(width 0)
+			(type default)
+		)
+	)
+	(wire
+		(pts
 			(xy 76.2 66.04) (xy 92.71 66.04)
 		)
@@
 	(bus
 		(pts
-			(xy 113.03 132.08) (xy 113.03 134.62)
+			(xy 114.3 132.08) (xy 114.3 134.62)
 		)
 		(stroke
@@
 	(bus
 		(pts
-			(xy 113.03 127) (xy 113.03 129.54)
+			(xy 114.3 127) (xy 114.3 129.54)
 		)
 		(stroke
@@
 	(bus
 		(pts
-			(xy 113.03 121.92) (xy 113.03 124.46)
+			(xy 114.3 121.92) (xy 114.3 124.46)
 		)
 		(stroke
@@
 	(wire
 		(pts
+			(xy 107.95 127) (xy 111.76 127)
+		)
+		(stroke
+			(width 0)
+			(type default)
+		)
+	)
+	(wire
+		(pts
 			(xy 53.34 96.52) (xy 71.12 96.52)
 		)
@@
 		)
 	)
+	(wire
+		(pts
+			(xy 107.95 121.92) (xy 111.76 121.92)
+		)
+		(stroke
+			(width 0)
+			(type default)
+		)
+	)
 	(bus
 		(pts
@@
 	(wire
 		(pts
-			(xy 107.95 124.46) (xy 110.49 124.46)
-		)
-		(stroke
-			(width 0)
-			(type default)
-		)
-	)
-	(wire
-		(pts
 			(xy 107.95 101.6) (xy 111.76 101.6)
 		)
@@
 	(bus
 		(pts
-			(xy 215.9 146.05) (xy 113.03 146.05)
+			(xy 215.9 142.24) (xy 114.3 142.24)
 		)
 		(stroke
@@
 	(bus
 		(pts
-			(xy 113.03 134.62) (xy 113.03 137.16)
-		)
-		(stroke
-			(width 0)
-			(type default)
-		)
-	)
-	(wire
-		(pts
-			(xy 107.95 134.62) (xy 110.49 134.62)
+			(xy 114.3 134.62) (xy 114.3 137.16)
 		)
 		(stroke
@@
 	(wire
 		(pts
-			(xy 107.95 137.16) (xy 110.49 137.16)
-		)
-		(stroke
-			(width 0)
-			(type default)
-		)
-	)
-	(wire
-		(pts
 			(xy 60.96 114.3) (xy 77.47 114.3)
 		)
@@
 	(wire
 		(pts
-			(xy 107.95 119.38) (xy 110.49 119.38)
+			(xy 107.95 119.38) (xy 111.76 119.38)
 		)
 		(stroke
@@
 	(bus
 		(pts
-			(xy 113.03 137.16) (xy 113.03 139.7)
+			(xy 114.3 137.16) (xy 114.3 139.7)
 		)
 		(stroke
@@
 	(bus
 		(pts
-			(xy 215.9 90.17) (xy 215.9 146.05)
+			(xy 215.9 90.17) (xy 215.9 142.24)
 		)
 		(stroke
@@
 		)
 	)
-	(text "To improve routing, address and data lines\nare arbitrarily assigned to the address and\ndata pins of the SRAM."
+	(text "To simplify routing, address\nand data lines are arbitrarily\nassigned to the address and\ndata pins of the SRAM."
 		(exclude_from_sim no)
-		(at 132.08 133.35 0)
+		(at 143.51 127 0)
 		(effects
 			(font
@@
 		)
 	)
-	(text "~{RES}, ~{IRQ}, and ~{NMI} are open-drain and wire ORed.\n\nRDY is bidirectional and wire ORed.\n\n~{SO} is pulled high by the FPGA."
+	(text "~{RES}, ~{IRQ}, ~{NMI}, and RDY are\nopen-drain and wire ORed.\n\n~{SO} is driven high by the FPGA."
 		(exclude_from_sim no)
-		(at 39.37 165.1 0)
+		(at 50.8 154.94 0)
 		(effects
 			(font
@@
 		)
 	)
-	(text "The bus is shared with the FPGA.  The FPGA deasserts BE (Bus Enable)\nto transition the CPU's Address, Data, and R~{W} buffers to high-Z\nwhile the FPGA drives the bus.\n\nCPU and RAM operate at +3V3 to interface directly with the FPGA.\nLevel shifters are used for connections to the 5V I/O section.\nThis split avoids needing level shifters for A[5..16]."
+	(text "CPU and RAM operate at 3V3 so that the system bus\nand CPU control signals can be directly shared\nwith the FPGA.\n\nLevel shifters are used for connections to the 5V\nI/O section.  This design avoids needing level\nshifters for A[5..16].\n\nThe FPGA deasserts BE (Bus Enable) to transition the\nCPU's Address, Data, and R~{W} buffers to high-Z\nwhen the FPGA drives the bus.\n\n"
 		(exclude_from_sim no)
-		(at 46.99 39.37 0)
+		(at 60.96 41.91 0)
 		(effects
 			(font

Commit message: hw: tidy schematics for publication
Other:
- company: (none) -> https://is.gd/6hpvh6
Changed lines of the file:
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@@
 		(date "2023-10-01")
 		(rev "A")
-		(comment 1 "Unspecified resistors are 1% and rated for 62.5mW or higher")
-		(comment 2 "Unspecified capacitors are rated for 25V or higher")
+		(company "https://is.gd/6hpvh6")
+		(comment 1 "Unspecified resistors are 1% / 62.5mW")
+		(comment 2 "Unspecified capacitors are 25V")
 		(comment 3 "Signals with B-prefix are level-shifted from 3V3 to 5V")
+		(comment 4 "License: CC0 1.0 Universal (Public Domain Dedication)")
 	)
 	(bus_alias "RAM_A"

Commit message: hw: schematic annotations
Other:
- note added: "A single 128 KB SRAM chip provides all memory regions: 32 KB main RAM, 64 KB expansion RAM (banked), 2 KB display RAM, 2 KB character ROM, and 26 KB system ROM. ROM contents are initialized by the MCU at power-on reset (POR) through an SPI-to-bus bridge implemented in the FPGA. Address lines A[15:0] form the shared system bus, connecting the CPU, I/O, FPGA, and most SRAM address pins. The excepti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"
- note added: "The CPU and RAM operate at 3V3, allowing the system bus and control signals to interface directly with the FPGA. Therefore, level shifters are only required where the CPU / FPGA interface with the 5 V I/O section. This avoids needing level shifters for A[5..16]. When the FPGA drives the bus, it deasserts BE (Bus Enable) to place the CPU's Address, Data, and R/~W buffers in a high-impedance state."
- note removed: "A single 128KB SRAM chip is used for the 32K main RAM, 64K expansion RAM, 2K display RAM, 2K character ROM and 26K system ROM. ROMs are initialized by the MCU on POR (via SPI -> bus bridge provided by the FPGA). A[15:0] are the address of the shared system bus, which is connected to the CPU, IO, FPGA and most RAM address pins. The exceptions are RAM_A[16:15,11:10], which are driven exclusively by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"
- note removed: "CPU and RAM operate at 3V3 so that the system bus and CPU control signals can be directly shared with the FPGA. Level shifters are used for connections to the 5V I/O section. This design avoids needing level shifters for A[5..16]. The FPGA deasserts BE (Bus Enable) to transition the CPU's Address, Data, and R~{W} buffers to high-Z when the FPGA drives the bus."
Changed lines of the file:
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@@
 		)
 	)
-	(text "A single 128KB SRAM chip is used for the 32K main RAM, 64K expansion RAM,\n2K display RAM, 2K character ROM and 26K system ROM.  ROMs are initialized\nby the MCU on POR (via SPI -> bus bridge provided by the FPGA).\n\nA[15:0] are the address of the shared system bus, which is connected to the\nCPU, IO, FPGA and most RAM address pins.  The exceptions are\nRAM_A[16:15,11:10], which are driven exclusively by the FPGA.\n\nRAM_A[11:10] is used by the FPGA to mirror display RAM when the CPU\naccesses the range $8000-8FFF.\n\n40 column PET has 1k of screen RAM, mirrored 4 times.\n80 column PET has 2k of screen RAM, mirrored 2 times.\n\nRAM_A[16:15] is used by the FPGA to implement bank switching when the\nCPU accesses the ranges $8000-FFFF.  The FPGA monitors writes to the\ncontrol register at $FFF0 to determine which bank is currently selected."
+	(text "A single 128 KB SRAM chip provides all memory regions: 32 KB main RAM,\n64 KB expansion RAM (banked), 2 KB display RAM, 2 KB character ROM,\nand 26 KB system ROM.\n\nROM contents are initialized by the MCU at power-on reset (POR) through\nan SPI-to-bus bridge implemented in the FPGA.\n\nAddress lines A[15:0] form the shared system bus, connecting the CPU,\nI/O, FPGA, and most SRAM address pins.  The exceptions are\nRAM_A[16:15, 11:10], which are routed through the FPGA instead of\nconnected directly to the bus.\n\nRAM_A[11:10] is used by the FPGA to mirror display RAM when the CPU\naccesses the range $8000-8FFF.\n\n40 column PET has 1k of screen RAM, mirrored 4 times.\n80 column PET has 2k of screen RAM, mirrored 2 times.\n\nThe FPGA uses RAM_A[16:15] to implement bank switching for CPU\naccesses in the range $8000-FFFF.  Writes to the control register at\n$FFF0 are monitored by the FPGA to determine the active bank.\n"
 		(exclude_from_sim no)
-		(at 176.53 55.88 0)
+		(at 171.45 58.42 0)
 		(effects
 			(font
@@
 		)
 	)
-	(text "CPU and RAM operate at 3V3 so that the system bus\nand CPU control signals can be directly shared\nwith the FPGA.\n\nLevel shifters are used for connections to the 5V\nI/O section.  This design avoids needing level\nshifters for A[5..16].\n\nThe FPGA deasserts BE (Bus Enable) to transition the\nCPU's Address, Data, and R~{W} buffers to high-Z\nwhen the FPGA drives the bus.\n\n"
+	(text "The CPU and RAM operate at 3V3, allowing the system\nbus and control signals to interface directly with\nthe FPGA.\n\nTherefore, level shifters are only required where\nthe CPU / FPGA interface with the 5 V I/O section.\nThis avoids needing level shifters for A[5..16].\n\nWhen the FPGA drives the bus, it deasserts BE\n(Bus Enable) to place the CPU's Address, Data, and\nR/~W buffers in a high-impedance state."
 		(exclude_from_sim no)
-		(at 60.96 41.91 0)
+		(at 58.42 39.37 0)
 		(effects
 			(font
