File: hw/rev-b/mainboard/kicad/FLASH.kicad_sch (KiCad schematic)
At the start: 5 parts, among them SW6 BOOTSEL, U22 W25Q128JVS

Commit message: cr(hw): use SMD push buttons
Parts:
- SW6: footprint EconoPET:SW_PUSH_1P1T_6x3.5mm_H4.3_APEM_MJTP1243 -> LCSC:SW-SMD_L3.9-W3.0-P4.45; LCSC (none) -> C720477
Changed lines of the file:
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@@
 			)
 		)
-		(property "Footprint" "EconoPET:SW_PUSH_1P1T_6x3.5mm_H4.3_APEM_MJTP1243"
+		(property "Footprint" "LCSC:SW-SMD_L3.9-W3.0-P4.45"
 			(at 116.84 107.95 0)
 			(effects
@@
 			)
 		)
-		(property "Datasheet" "~"
+		(property "Datasheet" "https://jlcpcb.com/api/file/downloadByFileSystemAccessId/8588886944068096000"
 			(at 116.84 107.95 0)
 			(effects
@@
 			)
 		)
-		(property "LCSC" ""
+		(property "LCSC" "C720477"
 			(at 121.92 107.95 90)
 			(effects
