File: hw/rev-b/mainboard/kicad/CPU.kicad_sch (KiCad schematic)
At the start: 12 parts, among them SW1 RESET, SW2 NMI, U1 W65C02S, U2 AS6C1008

Commit message: cr(hw): use SMD push buttons
Parts:
- SW1, SW2: footprint EconoPET:SW_PUSH_1P1T_6x3.5mm_H4.3_APEM_MJTP1243 -> LCSC:SW-SMD_L3.9-W3.0-P4.45; LCSC (none) -> C720477
Changed lines of the file:
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@@
 			)
 		)
-		(property "Footprint" "EconoPET:SW_PUSH_1P1T_6x3.5mm_H4.3_APEM_MJTP1243"
+		(property "Footprint" "LCSC:SW-SMD_L3.9-W3.0-P4.45"
 			(at 90.17 184.15 0)
 			(effects
@@
 			)
 		)
-		(property "Datasheet" "~"
+		(property "Datasheet" "https://jlcpcb.com/api/file/downloadByFileSystemAccessId/8588886944068096000"
 			(at 90.17 184.15 0)
 			(effects
@@
 		)
 		(property "MOUSER" "611-PTS636SK43LFS"
+			(at 95.25 184.15 0)
+			(effects
+				(font
+					(size 1.27 1.27)
+				)
+				(hide yes)
+			)
+		)
+		(property "LCSC" "C720477"
 			(at 95.25 184.15 0)
 			(effects
@@
 			)
 		)
-		(property "Footprint" "EconoPET:SW_PUSH_1P1T_6x3.5mm_H4.3_APEM_MJTP1243"
+		(property "Footprint" "LCSC:SW-SMD_L3.9-W3.0-P4.45"
 			(at 120.65 184.15 0)
 			(effects
@@
 			)
 		)
-		(property "Datasheet" "~"
+		(property "Datasheet" "https://jlcpcb.com/api/file/downloadByFileSystemAccessId/8588886944068096000"
 			(at 120.65 184.15 0)
 			(effects
@@
 			(at 125.73 184.15 0)
 			(effects
+				(font
+					(size 1.27 1.27)
+				)
+				(hide yes)
+			)
+		)
+		(property "LCSC" "C720477"
+			(at 125.73 184.15 0)
+			(effects

Commit message: pre-routing
Parts:
- U2: value AS6C1008 -> IS62WV1288BLL-55QLI; footprint Package_DIP:DIP-32_W15.24mm_Socket -> LCSC:SOP-32_L20.7-W11.3-P1.27-LS14.1-BL; LCSC (none) -> C1351025; MOUSER 913-AS6C1008-55PCN,649-DILB32P223TLF -> (none)
Other:
- note added: "128KB 55NS"
- note removed: "RAM 128KB"
Changed lines of the file:
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@@
 		)
 	)
-	(text " RAM\n128KB"
+	(text "128KB\n55NS"
 		(exclude_from_sim no)
-		(at 185.42 104.14 0)
-		(effects
-			(font
-				(size 1.27 1.27)
-			)
-			(justify left bottom)
+		(at 187.96 116.84 0)
+		(effects
+			(font
+				(size 1.27 1.27)
+			)
+			(justify bottom)
 		)
 	)
@@
 			)
 		)
-		(property "Value" "AS6C1008"
-			(at 187.96 96.52 0)
+		(property "Value" "IS62WV1288BLL-55QLI"
+			(at 187.96 96.52 90)
 			(effects
 				(font
@@
 			)
 		)
-		(property "Footprint" "Package_DIP:DIP-32_W15.24mm_Socket"
+		(property "Footprint" "LCSC:SOP-32_L20.7-W11.3-P1.27-LS14.1-BL"
 			(at 187.96 95.25 0)
 			(effects
@@
 			)
 		)
-		(property "Datasheet" "https://www.mouser.com/datasheet/2/12/AS6C1008feb2007-1511508.pdf"
+		(property "Datasheet" "https://www.lcsc.com/datasheet/C1351025.pdf"
 			(at 187.96 95.25 0)
 			(effects
@@
 			)
 		)
-		(property "MOUSER" "913-AS6C1008-55PCN,649-DILB32P223TLF"
+		(property "LCSC" "C1351025"
 			(at 187.96 97.79 0)
 			(effects
