File: hw/rev-b/mainboard/kicad/POWER.kicad_sch (KiCad schematic)
At the start: 79 parts, among them J10 5V PWR, J11 9V POWER, J13 9V POWER JACK, J27 6V POWER, J8 PET POWER, U3 AMS1117-3.3, U4 TPS5430DDA, U5 LM317AG-TN3-R, U6 TPS5430DDA

Commit message: hw: many touch ups
Parts:
- removed C117, C126, C15, C17, C89: 22u, Capacitor_SMD:C_0805_2012Metric, symbol Device:C_Small
- C110: value 330uF -> 2200uF; MOUSER 667-EEU-FM1V331 -> 232-25PK2200MEFC125X
- C111: value 15000uF -> 2200uF; MOUSER 661-BV250L153AM40S -> 232-25PK2200MEFC125X; now fitted
- C12: value 22u -> 47u 10V; footprint Capacitor_SMD:C_0805_2012Metric -> Capacitor_SMD:C_1206_3216Metric; LCSC C45783 -> C96123
Connections:
- net +5V: now also C12.2
- net +9V_Unreg: no longer C12.2

Commit message: hw: update qr-code for rev. B
Parts:
- SYM4: footprint Symbol:OSHW-Logo2_7.3x6mm_SilkScreen -> Symbol:OSHW-Logo2_9.8x8mm_SilkScreen
- SYM5: footprint EconoPET:EconoPET_QR -> EconoPET:EconoPET_QR_Rev_B
Changed lines of the file:
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@@
 			)
 		)
-		(property "Footprint" "Symbol:OSHW-Logo2_7.3x6mm_SilkScreen"
+		(property "Footprint" "Symbol:OSHW-Logo2_9.8x8mm_SilkScreen"
 			(at 19.05 39.37 0)
 			(effects
@@
 			)
 		)
-		(property "Footprint" "EconoPET:EconoPET_QR"
+		(property "Footprint" "EconoPET:EconoPET_QR_Rev_B"
 			(at 19.05 34.29 0)
 			(effects

Commit message: chore(hw): tidy and set ${REVISION} to "B"
Other:
- company: https://is.gd/6hpvh6 -> https://tinyurl.com/econopet-rev-b
Changed lines of the file:
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@@
 	(title_block
 		(title "EconoPET 40/8096")
-		(date "2026-02-27")
-		(rev "B")
-		(company "https://is.gd/6hpvh6")
+		(date "2026-08-25")
+		(rev "${REVISION}")
+		(company "https://tinyurl.com/econopet-rev-b")
 		(comment 1 "Unspecified resistors are 1% / 62.5mW")
 		(comment 2 "Unspecified capacitors are 25V")
