File: hw/rev-b/mainboard/kicad/CASS.kicad_sch (KiCad schematic)
At the start: 19 parts, among them J15 CASS_A_HEADER, J16 CASS_B_HEADER, J3 CASS_A_EDGE, J6 CASS_B_EDGE, Q2 AO3401A, Q3 AO3401A

Commit message: chore(hw): tidy and set ${REVISION} to "B"
Other:
- company: https://is.gd/6hpvh6 -> https://tinyurl.com/econopet-rev-b
Changed lines of the file:
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@@
 	(title_block
 		(title "EconoPET 40/8096")
-		(date "2026-02-27")
-		(rev "B")
-		(company "https://is.gd/6hpvh6")
+		(date "2026-08-25")
+		(rev "${REVISION}")
+		(company "https://tinyurl.com/econopet-rev-b")
 		(comment 1 "Unspecified resistors are 1% / 62.5mW")
 		(comment 2 "Unspecified capacitors are 25V")

Commit message: chore(hw): create production files
Parts:
- C77: LCSC C23733 -> (none); LCSC Part # (none) -> C23733
- D10, D9: LCSC C2286 -> (none); LCSC Part # (none) -> C2286
- J3, J6: now left out of the parts list
- Q2, Q3: FT Rotation Offset (none) -> 180; LCSC C15127 -> (none); LCSC Part # (none) -> C15127
- R32, R33: LCSC C25744 -> (none); LCSC Part # (none) -> C25744
- R34, R35: LCSC C25867 -> (none); LCSC Part # (none) -> C25867
