File: hw/rev-b/mainboard/kicad/IEEE.kicad_sch (KiCad schematic)
At the start: 26 parts, among them J1 IEEE_EDGE, J20 IEEE_HEADER, U14 SN74LS07, U15 SN74LS07, U16 SN74LS07, U17 74LS245, U18 74LS245

Commit message: chore(hw): tidy and set ${REVISION} to "B"
Other:
- company: https://is.gd/6hpvh6 -> https://tinyurl.com/econopet-rev-b
Changed lines of the file:
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@@
 	(title_block
 		(title "EconoPET 40/8096")
-		(date "2026-02-27")
-		(rev "B")
-		(company "https://is.gd/6hpvh6")
+		(date "2026-08-25")
+		(rev "${REVISION}")
+		(company "https://tinyurl.com/econopet-rev-b")
 		(comment 1 "Unspecified resistors are 1% / 62.5mW")
 		(comment 2 "Unspecified capacitors are 25V")

Commit message: chore(hw): create production files
Parts:
- C70, C71, C72, C73, C74: LCSC C307331 -> (none); LCSC Part # (none) -> C307331
- C75: LCSC C23733 -> (none); LCSC Part # (none) -> C23733
- J1: now left out of the parts list
- R30, R31: LCSC C25117 -> (none); LCSC Part # (none) -> C25117
- RN1, RN4, RN5, RN8: LCSC C29718 -> (none); LCSC Part # (none) -> C29718
- RN11, RN12, RN13: LCSC C25510 -> (none); LCSC Part # (none) -> C25510
- RN2, RN3, RN6, RN7: LCSC C1980 -> (none); LCSC Part # (none) -> C1980
- U14, U15, U16: LCSC C513513 -> (none); LCSC Part # (none) -> C513513
- U17, U18: LCSC C129580 -> (none); LCSC Part # (none) -> C129580
