File: hw/rev-b/mainboard/kicad/Keyboard.kicad_sch (KiCad schematic)
At the start: 7 parts, among them J19 KEYBOARD_EX, J5 KEYBOARD, U19 74LS145

Commit message: chore(hw): tidy and set ${REVISION} to "B"
Other:
- company: https://is.gd/6hpvh6 -> https://tinyurl.com/econopet-rev-b
Changed lines of the file:
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@@
 	(title_block
 		(title "EconoPET 40/8096")
-		(date "2026-02-27")
-		(rev "B")
-		(company "https://is.gd/6hpvh6")
+		(date "2026-08-25")
+		(rev "${REVISION}")
+		(company "https://tinyurl.com/econopet-rev-b")
 		(comment 1 "Unspecified resistors are 1% / 62.5mW")
 		(comment 2 "Unspecified capacitors are 25V")

Commit message: chore(hw): create production files
Parts:
- C78: LCSC C307331 -> (none); LCSC Part # (none) -> C307331
- C79: LCSC C23733 -> (none); LCSC Part # (none) -> C23733
- RN14, RN15: LCSC C29718 -> (none); LCSC Part # (none) -> C29718
- U19: LCSC C60829 -> (none); LCSC Part # (none) -> C60829
Changed lines of the file:
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@@
+			)
+		)
+		(property "FT Position Offset" ""
+			(at 201.93 73.66 0)
+			(effects
+				(font
+					(size 1.27 1.27)
+				)
+				(hide yes)
+			)
+		)
+		(property "FT Rotation Offset" ""
+			(at 201.93 73.66 0)
+			(effects
+				(font
+					(size 1.27 1.27)
+				)
+				(hide yes)
 			)
 		)
@@
 			)
 		)
-		(property "LCSC" "C307331"
+		(property "LCSC Part #" "C307331"
+			(at 93.98 54.61 0)
+			(effects
+				(font
+					(size 1.27 1.27)
+				)
+				(hide yes)
+			)
+		)
+		(property "FT Position Offset" ""
+			(at 93.98 54.61 0)
+			(effects
+				(font
+					(size 1.27 1.27)
+				)
+				(hide yes)
+			)
+		)
+		(property "FT Rotation Offset" ""
 			(at 93.98 54.61 0)
 			(effects
@@
 			)
 		)
-		(property "LCSC" "C60829"
+		(property "LCSC Part #" "C60829"
+			(at 110.49 78.74 0)
+			(effects
+				(font
+					(size 1.27 1.27)
+				)
+				(hide yes)
+			)
+		)
+		(property "FT Position Offset" ""
+			(at 110.49 78.74 0)
+			(effects
+				(font
+					(size 1.27 1.27)
+				)
+				(hide yes)
+			)
+		)
+		(property "FT Rotation Offset" ""
 			(at 110.49 78.74 0)
 			(effects
@@
 			)
 		)
+		(property "FT Position Offset" ""
+			(at 199.39 135.89 0)
+			(effects
+				(font
+					(size 1.27 1.27)
+				)
+				(hide yes)
+			)
+		)
+		(property "FT Rotation Offset" ""
+			(at 199.39 135.89 0)
+			(effects
+				(font
+					(size 1.27 1.27)
+				)
+				(hide yes)
+			)
+		)
 		(pin "1"
 		)
@@
 			)
 		)
-		(property "LCSC" "C23733"
+		(property "LCSC Part #" "C23733"
+			(at 229.87 133.35 0)
+			(effects
+				(font
+					(size 1.27 1.27)
+				)
+				(hide yes)
+			)
+		)
+		(property "FT Position Offset" ""
+			(at 229.87 133.35 0)
+			(effects
+				(font
+					(size 1.27 1.27)
+				)
+				(hide yes)
+			)
+		)
+		(property "FT Rotation Offset" ""
 			(at 229.87 133.35 0)
 			(effects
@@
 			)
 		)
-		(property "LCSC" "C29718"
+		(property "LCSC Part #" "C29718"
+			(at 154.94 40.64 0)
+			(effects
+				(font
+					(size 1.27 1.27)
+				)
+				(hide yes)
+			)
+		)
+		(property "FT Position Offset" ""
+			(at 154.94 40.64 0)
+			(effects
+				(font
+					(size 1.27 1.27)
+				)
+				(hide yes)
+			)
+		)
+		(property "FT Rotation Offset" ""
 			(at 154.94 40.64 0)
 			(effects
@@
 			)
 		)
-		(property "LCSC" "C29718"
+		(property "LCSC Part #" "C29718"
 			(at 172.72 40.64 0)
 			(effects
+				(font
+					(size 1.27 1.27)
+				)
+				(hide yes)
+			)
+		)
+		(property "FT Position Offset" ""
+			(at 172.72 40.64 0)
+			(effects
+				(font
+					(size 1.27 1.27)
+				)
+				(hide yes)
+			)
+		)
+		(property "FT Rotation Offset" ""
+			(at 172.72 40.64 0)
+			(effects
