File: hw/rev-b/mainboard/kicad/USB.kicad_sch (KiCad schematic)
At the start: 6 parts, among them J26 USB1.1_HOST_TYPE_C

Commit message: chore(hw): tidy and set ${REVISION} to "B"
Other:
- company: https://is.gd/6hpvh6 -> https://tinyurl.com/econopet-rev-b
Changed lines of the file:
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@@
 	(title_block
 		(title "EconoPET 40/8096")
-		(date "2026-02-27")
-		(rev "B")
-		(company "https://is.gd/6hpvh6")
+		(date "2026-08-25")
+		(rev "${REVISION}")
+		(company "https://tinyurl.com/econopet-rev-b")
 		(comment 1 "Unspecified resistors are 1% / 62.5mW")
 		(comment 2 "Unspecified capacitors are 25V")

Commit message: fix(hw): use TPS56424x for 5V / 6.1V rails (schematics only)
Other:
- note added: "USB 1.1 Host over USB-C connector The 56k pullups on CC1 and CC2 identify the port as downstream facing, supplying 5V/900ma. The diode prevents connected devices from inadvertently backpowering the EconoPET. V_{F} < 0.5V should be within USB spec of 5V +/-10% (4.5V - 5.5V). The 47u capacitor helps with current inrush (although hot insertion is not recommened.) Consider using an independently powe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"
- note removed: "USB 1.1 Host over USB-C connector The 56k pullups on CC1 and CC2 identify the port as downstream facing, supplying 5V/900ma. The diode prevents connected devices from inadvertently backpowering the EconoPET. V_{F} < 0.5V should be within USB spec of 5V +/-10%. The 47u capacitor helps with current inrush (although hot insertion is not recommened.) Consider using an independently powered USB hub as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"
Changed lines of the file:
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@@
 		)
 	)
-	(text "USB 1.1 Host over USB-C connector\n\nThe 56k pullups on CC1 and CC2 identify the\nport as downstream facing, supplying 5V/900ma.\n\nThe diode prevents connected devices from\ninadvertently backpowering the EconoPET.\n\nV_{F} < 0.5V should be within USB spec of\n5V +/-10%.\n\nThe 47u capacitor helps with current inrush\n(although hot insertion is not recommened.)\n\nConsider using an independently powered USB\nhub as an extra layer of protection.\n"
+	(text "USB 1.1 Host over USB-C connector\n\nThe 56k pullups on CC1 and CC2 identify the\nport as downstream facing, supplying 5V/900ma.\n\nThe diode prevents connected devices from\ninadvertently backpowering the EconoPET.\n\nV_{F} < 0.5V should be within USB spec of\n5V +/-10% (4.5V - 5.5V).\n\nThe 47u capacitor helps with current inrush\n(although hot insertion is not recommened.)\n\nConsider using an independently powered USB\nhub as an extra layer of protection.\n"
 		(exclude_from_sim no)
 		(at 95.25 137.16 0)

Commit message: chore(hw): create production files
Parts:
- C102: LCSC C96123 -> (none); LCSC Part # (none) -> C96123
- C103: LCSC C52923 -> (none); LCSC Part # (none) -> C52923
- D12: LCSC C22452 -> (none); LCSC Part # (none) -> C22452
- J26: FT Position Offset (none) -> 0,1.3335; LCSC C165948 -> (none); LCSC Part # (none) -> C165948
- R63, R64: LCSC C25796 -> (none); LCSC Part # (none) -> C25796
Changed lines of the file:
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@@
 			)
 		)
-		(property "LCSC" "C52923"
+		(property "LCSC Part #" "C52923"
+			(at 113.03 82.55 0)
+			(effects
+				(font
+					(size 1.27 1.27)
+				)
+				(hide yes)
+			)
+		)
+		(property "FT Position Offset" ""
+			(at 113.03 82.55 0)
+			(effects
+				(font
+					(size 1.27 1.27)
+				)
+				(hide yes)
+			)
+		)
+		(property "FT Rotation Offset" ""
 			(at 113.03 82.55 0)
 			(effects
@@
 			)
 		)
-		(property "LCSC" "C165948"
+		(property "LCSC Part #" "C165948"
+			(at 167.64 92.71 0)
+			(effects
+				(font
+					(size 1.27 1.27)
+				)
+				(hide yes)
+			)
+		)
+		(property "FT Position Offset" "0,1.3335"
+			(at 167.64 92.71 0)
+			(effects
+				(font
+					(size 1.27 1.27)
+				)
+				(hide yes)
+			)
+		)
+		(property "FT Rotation Offset" ""
 			(at 167.64 92.71 0)
 			(effects
@@
 			)
 		)
-		(property "LCSC" "C22452"
+		(property "LCSC Part #" "C22452"
+			(at 99.06 66.04 0)
+			(effects
+				(font
+					(size 1.27 1.27)
+				)
+				(hide yes)
+			)
+		)
+		(property "FT Position Offset" ""
+			(at 99.06 66.04 0)
+			(effects
+				(font
+					(size 1.27 1.27)
+				)
+				(hide yes)
+			)
+		)
+		(property "FT Rotation Offset" ""
 			(at 99.06 66.04 0)
 			(effects
@@
 			)
 		)
-		(property "LCSC" "C25796"
+		(property "LCSC Part #" "C25796"
+			(at 143.51 85.09 0)
+			(effects
+				(font
+					(size 1.27 1.27)
+				)
+				(hide yes)
+			)
+		)
+		(property "FT Position Offset" ""
+			(at 143.51 85.09 0)
+			(effects
+				(font
+					(size 1.27 1.27)
+				)
+				(hide yes)
+			)
+		)
+		(property "FT Rotation Offset" ""
 			(at 143.51 85.09 0)
 			(effects
@@
 			)
 		)
-		(property "LCSC" "C96123"
+		(property "LCSC Part #" "C96123"
+			(at 99.06 82.55 0)
+			(effects
+				(font
+					(size 1.27 1.27)
+				)
+				(hide yes)
+			)
+		)
+		(property "FT Position Offset" ""
+			(at 99.06 82.55 0)
+			(effects
+				(font
+					(size 1.27 1.27)
+				)
+				(hide yes)
+			)
+		)
+		(property "FT Rotation Offset" ""
 			(at 99.06 82.55 0)
 			(effects
@@
 			)
 		)
-		(property "LCSC" "C25796"
+		(property "LCSC Part #" "C25796"
 			(at 143.51 82.55 0)
 			(effects
+				(font
+					(size 1.27 1.27)
+				)
+				(hide yes)
+			)
+		)
+		(property "FT Position Offset" ""
+			(at 143.51 82.55 0)
+			(effects
+				(font
+					(size 1.27 1.27)
+				)
+				(hide yes)
+			)
+		)
+		(property "FT Rotation Offset" ""
+			(at 143.51 82.55 0)
+			(effects
