File: hw/rev-b/mainboard/kicad/MAGIC.kicad_sch (KiCad schematic)
At the start: 16 parts, among them U7 SN74LVC4245A, U8 SN74LVC4245A, U9 SN74LVC4245A

Commit message: hw: label JIFFY signal, tidy stitching
Connections:
- net BVSYNC renamed BJIFFY
- net VSYNC renamed JIFFY
Other:
- sheet FPGA ports: added JIFFY; removed VSYNC
Changed lines of the file:
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@@
 		)
 	)
-	(label "VSYNC"
+	(label "JIFFY"
 		(at 44.45 114.3 0)
 		(fields_autoplaced yes)
@@
 		)
 	)
-	(label "VSYNC"
+	(label "JIFFY"
 		(at 201.93 52.07 0)
 		(fields_autoplaced yes)
@@
 		)
 	)
-	(hierarchical_label "BVSYNC"
+	(hierarchical_label "BJIFFY"
 		(shape output)
 		(at 234.95 52.07 0)
@@
 			)
 		)
-		(pin "VSYNC" output
-			(at 52.07 114.3 180)
+		(pin "~{AUDIO_DET}" input
+			(at 52.07 119.38 180)
 			(effects
 				(font
@@
 			)
 		)
-		(pin "~{AUDIO_DET}" input
-			(at 52.07 119.38 180)
+		(pin "JIFFY" output
+			(at 52.07 114.3 180)
 			(effects
 				(font

Commit message: hw: many touch ups
Other:
- sheet FPGA ports: added SD_~{CS}; removed none
- sheet MCU ports: added SD_~{CS}; removed none
Changed lines of the file:
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@@
 	(wire
 		(pts
-			(xy 45.72 95.25) (xy 52.07 95.25)
+			(xy 45.72 97.79) (xy 52.07 97.79)
 		)
 		(stroke
@@
 	(wire
 		(pts
-			(xy 45.72 85.09) (xy 52.07 85.09)
+			(xy 45.72 87.63) (xy 52.07 87.63)
 		)
 		(stroke
@@
 	(wire
 		(pts
-			(xy 45.72 67.31) (xy 52.07 67.31)
+			(xy 45.72 69.85) (xy 52.07 69.85)
 		)
 		(stroke
@@
 	(wire
 		(pts
-			(xy 45.72 77.47) (xy 52.07 77.47)
+			(xy 45.72 80.01) (xy 52.07 80.01)
 		)
 		(stroke
@@
 	(wire
 		(pts
+			(xy 45.72 64.77) (xy 52.07 64.77)
+		)
+		(stroke
+			(width 0)
+			(type default)
+		)
+	)
+	(wire
+		(pts
 			(xy 208.28 20.32) (xy 218.44 20.32)
 		)
@@
 	(wire
 		(pts
-			(xy 45.72 97.79) (xy 52.07 97.79)
+			(xy 45.72 100.33) (xy 52.07 100.33)
 		)
 		(stroke
@@
 	(wire
 		(pts
-			(xy 52.07 111.76) (xy 44.45 111.76)
+			(xy 52.07 114.3) (xy 44.45 114.3)
 		)
 		(stroke
@@
 	(wire
 		(pts
-			(xy 45.72 119.38) (xy 52.07 119.38)
+			(xy 45.72 121.92) (xy 52.07 121.92)
 		)
 		(stroke
@@
 	(wire
 		(pts
-			(xy 45.72 69.85) (xy 52.07 69.85)
+			(xy 45.72 72.39) (xy 52.07 72.39)
 		)
 		(stroke
@@
 	(wire
 		(pts
-			(xy 45.72 121.92) (xy 52.07 121.92)
+			(xy 45.72 124.46) (xy 52.07 124.46)
 		)
 		(stroke
@@
 	(wire
 		(pts
-			(xy 52.07 114.3) (xy 44.45 114.3)
+			(xy 52.07 116.84) (xy 44.45 116.84)
 		)
 		(stroke
@@
 	(wire
 		(pts
-			(xy 52.07 109.22) (xy 44.45 109.22)
+			(xy 52.07 111.76) (xy 44.45 111.76)
 		)
 		(stroke
@@
 	(wire
 		(pts
-			(xy 45.72 74.93) (xy 52.07 74.93)
+			(xy 45.72 77.47) (xy 52.07 77.47)
 		)
 		(stroke
@@
 	(wire
 		(pts
-			(xy 52.07 106.68) (xy 44.45 106.68)
+			(xy 52.07 109.22) (xy 44.45 109.22)
 		)
 		(stroke
@@
 	(wire
 		(pts
-			(xy 45.72 82.55) (xy 52.07 82.55)
+			(xy 45.72 85.09) (xy 52.07 85.09)
 		)
 		(stroke
@@
 	(wire
 		(pts
-			(xy 45.72 90.17) (xy 52.07 90.17)
+			(xy 45.72 92.71) (xy 52.07 92.71)
 		)
 		(stroke
@@
 	(wire
 		(pts
-			(xy 45.72 92.71) (xy 52.07 92.71)
+			(xy 45.72 95.25) (xy 52.07 95.25)
 		)
 		(stroke
@@
 	)
 	(label "JIFFY"
-		(at 44.45 114.3 0)
+		(at 44.45 116.84 0)
 		(fields_autoplaced yes)
 		(effects
@@
 	)
 	(label "HORIZ"
-		(at 44.45 109.22 0)
+		(at 44.45 111.76 0)
 		(fields_autoplaced yes)
 		(effects
@@
 	)
 	(label "VERT"
-		(at 44.45 111.76 0)
+		(at 44.45 114.3 0)
 		(fields_autoplaced yes)
 		(effects
@@
 	)
 	(label "VIDEO"
-		(at 44.45 106.68 0)
+		(at 44.45 109.22 0)
 		(fields_autoplaced yes)
 		(effects
@@
 	(hierarchical_label "AUDIO"
 		(shape output)
-		(at 45.72 121.92 180)
+		(at 45.72 124.46 180)
 		(fields_autoplaced yes)
 		(effects
@@
 	(hierarchical_label "~{AUDIO_DET}"
 		(shape input)
-		(at 45.72 119.38 180)
+		(at 45.72 121.92 180)
 		(fields_autoplaced yes)
 		(effects
@@
 	(sheet
 		(at 52.07 25.4)
-		(size 30.48 99.06)
+		(size 30.48 101.6)
 		(fields_autoplaced yes)
 		(stroke
@@
 		)
 		(property "Sheetfile" "FPGA.kicad_sch"
-			(at 52.07 125.0446 0)
+			(at 52.07 127.5846 0)
 			(effects
 				(font
@@
 		)
 		(pin "VERT" output
-			(at 52.07 111.76 180)
+			(at 52.07 114.3 180)
 			(effects
 				(font
@@
 		)
 		(pin "HORIZ" output
-			(at 52.07 109.22 180)
+			(at 52.07 111.76 180)
 			(effects
 				(font
@@
 		)
 		(pin "VIDEO" output
-			(at 52.07 106.68 180)
+			(at 52.07 109.22 180)
 			(effects
 				(font
@@
 		)
 		(pin "I2C1_SDA" bidirectional
-			(at 52.07 74.93 180)
+			(at 52.07 77.47 180)
 			(effects
 				(font
@@
 		)
 		(pin "I2C1_SCL" input
-			(at 52.07 77.47 180)
+			(at 52.07 80.01 180)
 			(effects
 				(font
@@
 		)
 		(pin "~{SPI_ENA}" output
-			(at 52.07 82.55 180)
+			(at 52.07 85.09 180)
 			(effects
 				(font
@@
 		)
 		(pin "CEC" bidirectional
-			(at 52.07 85.09 180)
+			(at 52.07 87.63 180)
 			(effects
 				(font
@@
 		)
 		(pin "SWD" bidirectional
-			(at 52.07 92.71 180)
+			(at 52.07 95.25 180)
 			(effects
 				(font
@@
 		)
 		(pin "SWCLK" input
-			(at 52.07 90.17 180)
+			(at 52.07 92.71 180)
 			(effects
 				(font
@@
 		)
 		(pin "UART_TX" input
-			(at 52.07 95.25 180)
+			(at 52.07 97.79 180)
 			(effects
 				(font
@@
 		)
 		(pin "UART_RX" output
-			(at 52.07 97.79 180)
+			(at 52.07 100.33 180)
 			(effects
 				(font
@@
 		)
 		(pin "I2C0_SCL" input
-			(at 52.07 69.85 180)
+			(at 52.07 72.39 180)
 			(effects
 				(font
@@
 		)
 		(pin "I2C0_SDA" bidirectional
-			(at 52.07 67.31 180)
+			(at 52.07 69.85 180)
 			(effects
 				(font
@@
 		)
 		(pin "AUDIO" output
-			(at 52.07 121.92 180)
+			(at 52.07 124.46 180)
 			(effects
 				(font
@@
 		)
 		(pin "~{AUDIO_DET}" input
-			(at 52.07 119.38 180)
+			(at 52.07 121.92 180)
 			(effects
 				(font
@@
 		)
 		(pin "JIFFY" output
-			(at 52.07 114.3 180)
+			(at 52.07 116.84 180)
+			(effects
+				(font
+					(size 1.27 1.27)
+				)
+				(justify left)
+			)
+		)
+		(pin "SD_~{CS}" input
+			(at 52.07 64.77 180)
 			(effects
 				(font
@@
 	(sheet
 		(at 26.035 25.4)
-		(size 19.685 74.93)
+		(size 19.685 77.47)
 		(fields_autoplaced yes)
 		(stroke
@@
 		)
 		(property "Sheetfile" "MCU.kicad_sch"
-			(at 26.035 100.9146 0)
+			(at 26.035 103.4546 0)
 			(effects
 				(font
@@
 		)
 		(pin "I2C1_SCL" output
-			(at 45.72 77.47 0)
+			(at 45.72 80.01 0)
 			(effects
 				(font
@@
 		)
 		(pin "I2C1_SDA" bidirectional
-			(at 45.72 74.93 0)
+			(at 45.72 77.47 0)
 			(effects
 				(font
@@
 		)
 		(pin "~{SPI_ENA}" input
-			(at 45.72 82.55 0)
+			(at 45.72 85.09 0)
 			(effects
 				(font
@@
 		)
 		(pin "CEC" bidirectional
-			(at 45.72 85.09 0)
+			(at 45.72 87.63 0)
 			(effects
 				(font
@@
 		)
 		(pin "SWCLK" output
-			(at 45.72 90.17 0)
+			(at 45.72 92.71 0)
 			(effects
 				(font
@@
 		)
 		(pin "SWD" bidirectional
-			(at 45.72 92.71 0)
+			(at 45.72 95.25 0)
 			(effects
 				(font
@@
 		)
 		(pin "UART_TX" output
-			(at 45.72 95.25 0)
+			(at 45.72 97.79 0)
 			(effects
 				(font
@@
 		)
 		(pin "UART_RX" input
-			(at 45.72 97.79 0)
+			(at 45.72 100.33 0)
 			(effects
 				(font
@@
 		)
 		(pin "I2C0_SDA" bidirectional
-			(at 45.72 67.31 0)
+			(at 45.72 69.85 0)
 			(effects
 				(font
@@
 		)
 		(pin "I2C0_SCL" output
-			(at 45.72 69.85 0)
+			(at 45.72 72.39 0)
+			(effects
+				(font
+					(size 1.27 1.27)
+				)
+				(justify right)
+			)
+		)
+		(pin "SD_~{CS}" output
+			(at 45.72 64.77 0)
 			(effects
 				(font

Commit message: chore(hw): tidy and set ${REVISION} to "B"
Other:
- company: https://is.gd/6hpvh6 -> https://tinyurl.com/econopet-rev-b
Changed lines of the file:
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@@
 	(title_block
 		(title "EconoPET 40/8096")
-		(date "2026-02-27")
-		(rev "B")
-		(company "https://is.gd/6hpvh6")
+		(date "2026-08-25")
+		(rev "${REVISION}")
+		(company "https://tinyurl.com/econopet-rev-b")
 		(comment 1 "Unspecified resistors are 1% / 62.5mW")
 		(comment 2 "Unspecified capacitors are 25V")

Commit message: chore(hw): create production files
Parts:
- C32: LCSC C23733 -> (none); LCSC Part # (none) -> C23733
- C33, C34, C35, C36, C37, C38: LCSC C307331 -> (none); LCSC Part # (none) -> C307331
- R18, R19, R20: LCSC C25744 -> (none); LCSC Part # (none) -> C25744
- R21, R22, R23: LCSC C25908 -> (none); LCSC Part # (none) -> C25908
- U7, U8, U9: LCSC C7859 -> (none); LCSC Part # (none) -> C7859

Commit message: feat(hw): separate audio_l / audio_r (schematic only)
Other:
- sheet FPGA ports: added AUDIO_L, AUDIO_R; removed AUDIO
Changed lines of the file:
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@@
 	(wire
 		(pts
+			(xy 45.72 127) (xy 52.07 127)
+		)
+		(stroke
+			(width 0)
+			(type default)
+		)
+	)
+	(wire
+		(pts
 			(xy 45.72 57.15) (xy 52.07 57.15)
 		)
@@
 		)
 	)
-	(hierarchical_label "AUDIO"
+	(hierarchical_label "AUDIO_L"
 		(shape output)
 		(at 45.72 124.46 180)
@@
 		)
 	)
+	(hierarchical_label "AUDIO_R"
+		(shape output)
+		(at 45.72 127 180)
+		(fields_autoplaced yes)
+		(effects
+			(font
+				(size 1.27 1.27)
+			)
+			(justify right)
+		)
+	)
 	(hierarchical_label "~{AUDIO_DET}"
 		(shape input)
@@
 	(sheet
 		(at 52.07 25.4)
-		(size 30.48 101.6)
+		(size 30.48 104.14)
 		(fields_autoplaced yes)
 		(stroke
@@
 		)
 		(property "Sheetfile" "FPGA.kicad_sch"
-			(at 52.07 127.5846 0)
+			(at 52.07 130.1246 0)
 			(effects
 				(font
@@
 			)
 		)
-		(pin "AUDIO" output
-			(at 52.07 124.46 180)
+		(pin "~{AUDIO_DET}" input
+			(at 52.07 121.92 180)
 			(effects
 				(font
@@
 			)
 		)
-		(pin "~{AUDIO_DET}" input
-			(at 52.07 121.92 180)
+		(pin "JIFFY" output
+			(at 52.07 116.84 180)
 			(effects
 				(font
@@
 			)
 		)
-		(pin "JIFFY" output
-			(at 52.07 116.84 180)
+		(pin "SD_~{CS}" input
+			(at 52.07 64.77 180)
 			(effects
 				(font
@@
 			)
 		)
-		(pin "SD_~{CS}" input
-			(at 52.07 64.77 180)
+		(pin "AUDIO_L" output
+			(at 52.07 124.46 180)
+			(effects
+				(font
+					(size 1.27 1.27)
+				)
+				(justify left)
+			)
+		)
+		(pin "AUDIO_R" output
+			(at 52.07 127 180)
 			(effects
 				(font
