File: hw/rev-b/mainboard/kicad/FPGA.kicad_sch (KiCad schematic)
At the start: 46 parts, among them J17 PMOD1, J18 PMOD2, J22 PROG, J4 BUS_EXPANSION, J9 FPGA_MCU, Q1 MMBT3904, SW3 CONFIG, U10 T20Q144C3

Commit message: hw: label JIFFY signal, tidy stitching
Connections:
- net VSYNC renamed JIFFY
Changed lines of the file:
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@@
 		)
 	)
-	(label "VSYNC"
+	(label "JIFFY"
 		(at 246.38 86.36 180)
 		(fields_autoplaced yes)
@@
 		)
 	)
-	(hierarchical_label "VSYNC"
+	(hierarchical_label "JIFFY"
 		(shape output)
 		(at 368.3 137.16 180)

Commit message: hw: many touch ups
Connections:
- net GND: no longer J9.14 (Pin_14)
- new net SD_~{CS}: J9.14 (Pin_14)
Other:
- moved on the sheet: C62
Changed lines of the file:
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@@
 	)
 	(junction
-		(at 229.87 58.42)
-		(diameter 0)
-		(color 0 0 0 0)
-	)
-	(junction
 		(at 361.95 101.6)
 		(diameter 0)
@@
 	(wire
 		(pts
+			(xy 217.17 58.42) (xy 231.14 58.42)
+		)
+		(stroke
+			(width 0)
+			(type default)
+		)
+	)
+	(wire
+		(pts
 			(xy 95.25 208.28) (xy 100.33 208.28)
 		)
@@
 		)
 	)
-	(wire
-		(pts
-			(xy 229.87 43.18) (xy 229.87 48.26)
-		)
-		(stroke
-			(width 0)
-			(type default)
-		)
-	)
 	(bus
 		(pts
@@
 	(wire
 		(pts
-			(xy 229.87 58.42) (xy 231.14 58.42)
-		)
-		(stroke
-			(width 0)
-			(type default)
-		)
-	)
-	(wire
-		(pts
 			(xy 22.86 63.5) (xy 22.86 64.77)
 		)
@@
 	(wire
 		(pts
-			(xy 229.87 53.34) (xy 229.87 58.42)
-		)
-		(stroke
-			(width 0)
-			(type default)
-		)
-	)
-	(wire
-		(pts
 			(xy 55.88 167.64) (xy 55.88 172.72)
 		)
@@
 	(wire
 		(pts
-			(xy 217.17 58.42) (xy 229.87 58.42)
-		)
-		(stroke
-			(width 0)
-			(type default)
-		)
-	)
-	(wire
-		(pts
 			(xy 53.34 29.21) (xy 55.88 29.21)
 		)
@@
 	(wire
 		(pts
+			(xy 229.87 44.45) (xy 229.87 43.18)
+		)
+		(stroke
+			(width 0)
+			(type default)
+		)
+	)
+	(wire
+		(pts
 			(xy 62.23 160.02) (xy 63.5 160.02)
 		)
@@
 		)
 	)
+	(hierarchical_label "SD_~{CS}"
+		(shape input)
+		(at 231.14 58.42 0)
+		(fields_autoplaced yes)
+		(effects
+			(font
+				(size 1.27 1.27)
+			)
+			(justify left)
+		)
+	)
 	(hierarchical_label "SPI1_~{READY}"
 		(shape output)
@@
 	(symbol
 		(lib_id "Device:C_Small")
-		(at 229.87 50.8 0)
+		(at 229.87 46.99 0)
 		(unit 1)
 		(exclude_from_sim no)
@@
 		(dnp no)
 		(property "Reference" "C62"
-			(at 232.2068 49.6316 0)
+			(at 232.2068 45.8216 0)
 			(effects
 				(font
@@
 		)
 		(property "Value" "4u7 10V"
-			(at 232.2068 51.943 0)
+			(at 232.2068 48.133 0)
 			(effects
 				(font
@@
 		)
 		(property "Footprint" "Capacitor_SMD:C_0402_1005Metric"
-			(at 229.87 50.8 0)
+			(at 229.87 46.99 0)
 			(effects
 				(font
@@
 		)
 		(property "Datasheet" "https://product.samsungsem.com/mlcc/CL05A475MP5NRN.do"
-			(at 229.87 50.8 0)
+			(at 229.87 46.99 0)
 			(effects
 				(font
@@
 		)
 		(property "Description" ""
-			(at 229.87 50.8 0)
+			(at 229.87 46.99 0)
 			(effects
 				(font
@@
 		)
 		(property "LCSC" "C23733"
-			(at 229.87 50.8 0)
+			(at 229.87 46.99 0)
 			(effects
 				(font
@@
 	(symbol
 		(lib_id "power:GND")
-		(at 231.14 58.42 90)
-		(mirror x)
+		(at 229.87 49.53 0)
+		(mirror y)
 		(unit 1)
 		(exclude_from_sim no)
@@
 		(dnp no)
 		(property "Reference" "#PWR070"
-			(at 237.49 58.42 0)
+			(at 229.87 55.88 0)
 			(effects
 				(font
@@
 		)
 		(property "Value" "GND"
-			(at 236.22 58.42 0)
+			(at 229.87 54.61 0)
 			(effects
 				(font
@@
 		)
 		(property "Footprint" ""
-			(at 231.14 58.42 0)
+			(at 229.87 49.53 0)
 			(effects
 				(font
@@
 		)
 		(property "Datasheet" ""
-			(at 231.14 58.42 0)
+			(at 229.87 49.53 0)
 			(effects
 				(font
@@
 		)
 		(property "Description" "Power symbol creates a global label with name \"GND\" , ground"
-			(at 231.14 58.42 0)
+			(at 229.87 49.53 0)
 			(effects
 				(font

Commit message: chore(hw): tidy and set ${REVISION} to "B"
Other:
- company: https://is.gd/6hpvh6 -> https://tinyurl.com/econopet-rev-b
Changed lines of the file:
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@@
 	(title_block
 		(title "EconoPET 40/8096")
-		(date "2026-02-27")
-		(rev "B")
-		(company "https://is.gd/6hpvh6")
+		(date "2026-08-25")
+		(rev "${REVISION}")
+		(company "https://tinyurl.com/econopet-rev-b")
 		(comment 1 "Unspecified resistors are 1% / 62.5mW")
 		(comment 2 "Unspecified capacitors are 25V")

Commit message: chore(hw): create production files
Parts:
- C39, C41, C42, C43: LCSC C52923 -> (none); LCSC Part # (none) -> C52923
- C40, C44, C45, C46, C47, C48, C49, C50, C51, C52, C53, C55, C57, C59: LCSC C307331 -> (none); LCSC Part # (none) -> C307331
- C54, C56, C58, C60, C61: LCSC C15195 -> (none); LCSC Part # (none) -> C15195
- C62, C63, C64, C65, C66: LCSC C23733 -> (none); LCSC Part # (none) -> C23733
- D7: LCSC C2986059 -> (none); LCSC Part # (none) -> C2986059
- D8: LCSC C2286 -> (none); LCSC Part # (none) -> C2286
- Q1: LCSC C20526 -> (none); LCSC Part # (none) -> C20526
- R24, R28: LCSC C25741 -> (none); LCSC Part # (none) -> C25741
- R25: LCSC C25744 -> (none); LCSC Part # (none) -> C25744
- R26: LCSC C25752 -> (none); LCSC Part # (none) -> C25752
- R27, R29: LCSC C11702 -> (none); LCSC Part # (none) -> C11702
- RN10, RN9: LCSC C29718 -> (none); LCSC Part # (none) -> C29718
- U10: LCSC C3278392 -> (none); LCSC Part # (none) -> C3278392

Commit message: feat(hw): separate audio_l / audio_r (schematic only)
Connections:
- net AUDIO renamed AUDIO_L
- net CSI renamed AUDIO_R
Other:
- moved on the sheet: C40, R24, U10A

Commit message: feat(hw): add config sw for refresh rate, tidy audio gnd fills
Parts:
- SW3: footprint EconoPET:SW_DIP_SPSTx02_Slide_6.7x6.64mm_W7.62mm_P2.54mm_LowProfile_or_SolderJumper -> EconoPET:SW_DIP_SPSTx03_Slide_6.7x9.18mm_W7.62mm_P2.54mm_LowProfile_or_SolderJumper; symbol Switch:SW_DIP_x02 -> Switch:SW_DIP_x03
Connections:
- net GND: now also J4.49 (Pin_49), J4.50 (Pin_50), SW3.3
- net S1: now also SW3.6; no longer SW3.4
- net S2: now also SW3.5; no longer SW3.3
- net ~{AUDIO_DET}: now also U10.20 (GPIOL_12_CDI2); no longer J4.50 (Pin_50), U10.19 (GPIOL_13_CDI3)
- removed net L12: J4.49 (Pin_49), U10.20 (GPIOL_12_CDI2)
- new net S3: SW3.4, U10.19 (GPIOL_13_CDI3)
Changed lines of the file:
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@@
 	)
 	(junction
-		(at 384.81 203.2)
-		(diameter 0)
-		(color 0 0 0 0)
-	)
-	(junction
 		(at 125.73 251.46)
 		(diameter 0)
@@
 	)
 	(junction
+		(at 382.27 149.86)
+		(diameter 0)
+		(color 0 0 0 0)
+	)
+	(junction
 		(at 120.65 233.68)
 		(diameter 0)
@@
 	)
 	(junction
+		(at 386.08 203.2)
+		(diameter 0)
+		(color 0 0 0 0)
+	)
+	(junction
 		(at 95.25 208.28)
 		(diameter 0)
@@
 	(wire
 		(pts
+			(xy 375.92 149.86) (xy 382.27 149.86)
+		)
+		(stroke
+			(width 0)
+			(type default)
+		)
+	)
+	(wire
+		(pts
 			(xy 95.25 203.2) (xy 95.25 205.74)
 		)
@@
 	(wire
 		(pts
-			(xy 383.54 203.2) (xy 384.81 203.2)
+			(xy 383.54 203.2) (xy 386.08 203.2)
 		)
 		(stroke
@@
 	(wire
 		(pts
+			(xy 388.62 203.2) (xy 388.62 201.93)
+		)
+		(stroke
+			(width 0)
+			(type default)
+		)
+	)
+	(wire
+		(pts
 			(xy 62.23 252.73) (xy 62.23 251.46)
 		)
@@
 	(wire
 		(pts
+			(xy 386.08 203.2) (xy 388.62 203.2)
+		)
+		(stroke
+			(width 0)
+			(type default)
+		)
+	)
+	(wire
+		(pts
 			(xy 154.94 142.24) (xy 129.54 142.24)
 		)
@@
 	(wire
 		(pts
+			(xy 144.78 121.92) (xy 149.86 121.92)
+		)
+		(stroke
+			(width 0)
+			(type default)
+		)
+	)
+	(wire
+		(pts
 			(xy 205.74 144.78) (xy 210.82 144.78)
 		)
@@
 	(wire
 		(pts
+			(xy 375.92 147.32) (xy 375.92 149.86)
+		)
+		(stroke
+			(width 0)
+			(type default)
+		)
+	)
+	(wire
+		(pts
 			(xy 151.13 251.46) (xy 151.13 252.73)
 		)
@@
 	(wire
 		(pts
-			(xy 384.81 203.2) (xy 386.08 203.2)
-		)
-		(stroke
-			(width 0)
-			(type default)
-		)
-	)
-	(wire
-		(pts
 			(xy 204.47 58.42) (xy 193.04 58.42)
 		)
@@
 	(wire
 		(pts
+			(xy 388.62 149.86) (xy 388.62 147.32)
+		)
+		(stroke
+			(width 0)
+			(type default)
+		)
+	)
+	(wire
+		(pts
 			(xy 50.8 29.21) (xy 50.8 30.48)
 		)
@@
 	(wire
 		(pts
+			(xy 382.27 149.86) (xy 388.62 149.86)
+		)
+		(stroke
+			(width 0)
+			(type default)
+		)
+	)
+	(wire
+		(pts
 			(xy 19.05 233.68) (xy 31.75 233.68)
 		)
@@
 	(wire
 		(pts
-			(xy 407.67 148.59) (xy 407.67 114.3)
+			(xy 407.67 152.4) (xy 407.67 114.3)
 		)
 		(stroke
@@
 		)
 	)
-	(label "L12"
-		(at 149.86 121.92 180)
+	(label "S3"
+		(at 149.86 124.46 180)
 		(fields_autoplaced yes)
 		(effects
@@
 		)
 	)
+	(label "S3"
+		(at 388.62 186.69 90)
+		(fields_autoplaced yes)
+		(effects
+			(font
+				(size 1.27 1.27)
+			)
+			(justify left bottom)
+		)
+	)
 	(label "A3"
 		(at 208.28 189.23 0)
@@
 		)
 	)
-	(label "L12"
-		(at 375.92 147.32 180)
-		(fields_autoplaced yes)
-		(effects
-			(font
-				(size 1.27 1.27)
-			)
-			(justify right bottom)
-		)
-	)
 	(label "A5"
 		(at 375.92 116.84 180)
@@
 	(hierarchical_label "~{AUDIO_DET}"
 		(shape input)
-		(at 149.86 124.46 180)
+		(at 144.78 121.92 180)
 		(fields_autoplaced yes)
 		(effects
@@
 		)
 	)
-	(hierarchical_label "~{AUDIO_DET}"
-		(shape input)
-		(at 388.62 147.32 0)
-		(fields_autoplaced yes)
-		(effects
-			(font
-				(size 1.27 1.27)
-			)
-			(justify left)
-		)
-	)
 	(hierarchical_label "SD_~{CS}"
 		(shape input)
@@
 	(symbol
 		(lib_id "power:GND")
-		(at 384.81 203.2 0)
+		(at 386.08 203.2 0)
 		(unit 1)
 		(exclude_from_sim no)
@@
 		(dnp no)
 		(property "Reference" "#PWR079"
-			(at 384.81 209.55 0)
+			(at 386.08 209.55 0)
 			(effects
 				(font
@@
 		)
 		(property "Value" "GND"
-			(at 384.81 207.645 0)
+			(at 386.08 207.645 0)
 			(effects
 				(font
@@
 		)
 		(property "Footprint" ""
-			(at 384.81 203.2 0)
+			(at 386.08 203.2 0)
 			(effects
 				(font
@@
 		)
 		(property "Datasheet" ""
-			(at 384.81 203.2 0)
+			(at 386.08 203.2 0)
 			(effects
 				(font
@@
 		)
 		(property "Description" "Power symbol creates a global label with name \"GND\" , ground"
-			(at 384.81 203.2 0)
+			(at 386.08 203.2 0)
 			(effects
 				(font
@@
 	)
 	(symbol
+		(lib_id "power:GND")
+		(at 382.27 149.86 0)
+		(mirror y)
+		(unit 1)
+		(exclude_from_sim no)
+		(in_bom yes)
+		(on_board yes)
+		(dnp no)
+		(property "Reference" "#PWR026"
+			(at 382.27 156.21 0)
+			(effects
+				(font
+					(size 1.27 1.27)
+				)
+				(hide yes)
+			)
+		)
+		(property "Value" "GND"
+			(at 382.143 154.2542 0)
+			(effects
+				(font
+					(size 1.27 1.27)
+				)
+			)
+		)
+		(property "Footprint" ""
+			(at 382.27 149.86 0)
+			(effects
+				(font
+					(size 1.27 1.27)
+				)
+				(hide yes)
+			)
+		)
+		(property "Datasheet" ""
+			(at 382.27 149.86 0)
+			(effects
+				(font
+					(size 1.27 1.27)
+				)
+				(hide yes)
+			)
+		)
+		(property "Description" "Power symbol creates a global label with name \"GND\" , ground"
+			(at 382.27 149.86 0)
+			(effects
+				(font
+					(size 1.27 1.27)
+				)
+				(hide yes)
+			)
+		)
+		(pin "1"
+		)
+		(instances
+			(project "Mainboard"
+				(path "/2eea20e6-112c-411a-b615-885ae773135a/00000000-0000-0000-0000-0000617d6918/00000000-0000-0000-0000-000062edbe39"
+					(reference "#PWR026")
+					(unit 1)
+				)
+			)
+		)
+	)
+	(symbol
 		(lib_id "Device:C_Small")
 		(at 87.63 255.27 0)
@@
 	)
 	(symbol
-		(lib_id "Switch:SW_DIP_x02")
+		(lib_id "Switch:SW_DIP_x03")
 		(at 386.08 194.31 90)
 		(unit 1)
@@
 		(on_board yes)
 		(dnp no)
-		(fields_autoplaced yes)
 		(property "Reference" "SW3"
 			(at 392.43 193.0399 90)
@@
 			)
 		)
-		(property "Footprint" "EconoPET:SW_DIP_SPSTx02_Slide_6.7x6.64mm_W7.62mm_P2.54mm_LowProfile_or_SolderJumper"
-			(at 386.08 194.31 0)
+		(property "Footprint" "EconoPET:SW_DIP_SPSTx03_Slide_6.7x9.18mm_W7.62mm_P2.54mm_LowProfile_or_SolderJumper"
+			(at 388.62 194.31 0)
 			(effects
 				(font
@@
 		)
 		(property "Datasheet" "~"
-			(at 386.08 194.31 0)
+			(at 388.62 194.31 0)
 			(effects
 				(font
@@
 			)
 		)
-		(property "Description" ""
+		(property "Description" "3x DIP Switch, Single Pole Single Throw (SPST) switch, small symbol"
 			(at 386.08 194.31 0)
 			(effects
@@
 		(pin "4"
 		)
+		(pin "5"
+		)
+		(pin "6"
+		)
 		(instances
 			(project ""
@@
 	(symbol
 		(lib_id "power:GND")
-		(at 407.67 148.59 0)
+		(at 407.67 152.4 0)
 		(mirror y)
 		(unit 1)
@@
 		(dnp no)
 		(property "Reference" "#PWR085"
-			(at 407.67 154.94 0)
+			(at 407.67 158.75 0)
 			(effects
 				(font
@@
 		)
 		(property "Value" "GND"
-			(at 407.543 152.9842 0)
+			(at 407.543 156.7942 0)
 			(effects
 				(font
@@
 		)
 		(property "Footprint" ""
-			(at 407.67 148.59 0)
+			(at 407.67 152.4 0)
 			(effects
 				(font
@@
 		)
 		(property "Datasheet" ""
-			(at 407.67 148.59 0)
+			(at 407.67 152.4 0)
 			(effects
 				(font
@@
 		)
 		(property "Description" "Power symbol creates a global label with name \"GND\" , ground"
-			(at 407.67 148.59 0)
+			(at 407.67 152.4 0)
 			(effects
 				(font
