File: hw/rev-b/mainboard/kicad/IO.kicad_sch (KiCad schematic)
At the start: 7 parts, among them U11 W65C21N, U12 W65C21N, U13 W65C22N

Commit message: hw: label JIFFY signal, tidy stitching
Parts:
- R38: value 470 -> 1k; LCSC C25117 -> C11702
Connections:
- net BVSYNC renamed BJIFFY
Other:
- note added: "1K protects VIA from "Killer Poke", which puts PB5 in contention with BJIFFY. W65C22N drives 1 CMOS load (~3ma). BJIFFY is driven at ~24ma by level shifter. (BJIFFY easily wins against VIA.)"
- note added: "In the original PET, both PIA1 CB1 and VIA PB5 were connected to VERT_DRIVE. PIA CB1 is an input only, and generates the 50/60 Hz jiffy interrupt. VIA PB5 was intended for detecting when the display was in vertical blank, but was also used as an output in the infamous "killer poke" trick. In our design, we replace VERT_DRIVE with an independently generated JIFFY clock. Typically, these signals wi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"
- note removed: "470R protects VIA from "Killer Poke", which puts PB5 in contention with BVERT. W65C22N drives 1 CMOS load (~3ma). BVERT is driven at ~24ma by level shifter. (BVERT easily wins against VIA.)"
- note removed: "VSYNC connects to both PIA1 CB1 and VIA PB5. PIA CB1 is an input only, and generates the 50/60 Hz Jiffy interrupt. VIA PB5 exposes the vertical sync signal as a normal GPIO input. Software can poll PB5 to determine whether the display is currently in vertical blank. This is what the ROM editor does before writing to screen RAM on early PETs to avoid "snow." It is also the signal used by the famou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"
Changed lines of the file:
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@@
 		)
 	)
-	(text "470R protects VIA from \"Killer Poke\", which\nputs PB5 in contention with BVERT.\n\nW65C22N drives 1 CMOS load (~3ma).\nBVERT is driven at ~24ma by level shifter.\n(BVERT easily wins against VIA.)\n"
+	(text "1K protects VIA from \"Killer Poke\", which\nputs PB5 in contention with BJIFFY.\n\nW65C22N drives 1 CMOS load (~3ma).\nBJIFFY is driven at ~24ma by level shifter.\n(BJIFFY easily wins against VIA.)\n"
 		(exclude_from_sim no)
 		(at 219.71 153.67 0)
@@
 		)
 	)
-	(text "VSYNC connects to both PIA1 CB1 and VIA PB5.\n\nPIA CB1 is an input only, and generates the 50/60 Hz Jiffy interrupt.\nVIA PB5 exposes the vertical sync signal as a normal GPIO input. Software\ncan poll PB5 to determine whether the display is currently in vertical blank.\nThis is what the ROM editor does before writing to screen RAM on early PETs\nto avoid \"snow.\" It is also the signal used by the famous \"killer poke\" trick."
+	(text "In the original PET, both PIA1 CB1 and VIA PB5 were connected to VERT_DRIVE.\nPIA CB1 is an input only, and generates the 50/60 Hz jiffy interrupt.\nVIA PB5 was intended for detecting when the display was in vertical blank,\nbut was also used as an output in the infamous \"killer poke\" trick.\n\nIn our design, we replace VERT_DRIVE with an independently generated JIFFY\nclock.  Typically, these signals will be identical, but generating them\nseparately affords the option of supporting a 60 Hz refresh rate with a\n50 Hz interrupt and vice-versa."
 		(exclude_from_sim no)
-		(at 151.13 59.69 0)
+		(at 151.13 57.15 0)
 		(effects
 			(font
@@
 		)
 	)
-	(hierarchical_label "BVSYNC"
+	(hierarchical_label "BJIFFY"
 		(shape input)
 		(at 240.03 68.58 0)
@@
 			)
 		)
-		(property "Value" "470"
+		(property "Value" "1k"
 			(at 229.108 140.462 90)
 			(effects
@@
 			)
 		)
-		(property "Datasheet" "https://www.lcsc.com/datasheet/lcsc_datasheet_2205311900_UNI-ROYAL-Uniroyal-Elec-0402WGF4700TCE_C25117.pdf"
+		(property "Datasheet" "https://www.lcsc.com/datasheet/lcsc_datasheet_2206010216_UNI-ROYAL-Uniroyal-Elec-0402WGF1001TCE_C11702.pdf"
 			(at 227.33 143.51 0)
 			(effects
@@
 			)
 		)
-		(property "LCSC" "C25117"
+		(property "LCSC" "C11702"
 			(at 227.33 143.51 0)
 			(effects

Commit message: hw: additional annotations for jiffy clock signal
Other:
- note added: "In the original PET, both PIA1 CB1 and VIA PB5 were connected to VERT_DRIVE. PIA CB1 is an input only, and generates the 50/60 Hz jiffy interrupt. VIA PB5 is a GPIO, typically configured as an input, and intended for detecting when the display was in vertical blank, but was also used as an output in the infamous "killer poke" trick. In our design, we replace VERT_DRIVE with an independently gener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"
- note removed: "In the original PET, both PIA1 CB1 and VIA PB5 were connected to VERT_DRIVE. PIA CB1 is an input only, and generates the 50/60 Hz jiffy interrupt. VIA PB5 was intended for detecting when the display was in vertical blank, but was also used as an output in the infamous "killer poke" trick. In our design, we replace VERT_DRIVE with an independently generated JIFFY clock. Typically, these signals wi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"
Changed lines of the file:
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@@
 		)
 	)
-	(text "In the original PET, both PIA1 CB1 and VIA PB5 were connected to VERT_DRIVE.\nPIA CB1 is an input only, and generates the 50/60 Hz jiffy interrupt.\nVIA PB5 was intended for detecting when the display was in vertical blank,\nbut was also used as an output in the infamous \"killer poke\" trick.\n\nIn our design, we replace VERT_DRIVE with an independently generated JIFFY\nclock.  Typically, these signals will be identical, but generating them\nseparately affords the option of supporting a 60 Hz refresh rate with a\n50 Hz interrupt and vice-versa."
+	(text "In the original PET, both PIA1 CB1 and VIA PB5 were connected to VERT_DRIVE.\nPIA CB1 is an input only, and generates the 50/60 Hz jiffy interrupt.\nVIA PB5 is a GPIO, typically configured as an input, and intended for detecting\nwhen the display was in vertical blank, but was also used as an output in the\ninfamous \"killer poke\" trick.\n\nIn our design, we replace VERT_DRIVE with an independently generated JIFFY\nclock.  Typically, JIFFY and VERT_DRIVE are identical, but generating them\nseparately affords the option of supporting a 60 Hz refresh rate with a\n50 Hz jiffy interrupt and vice-versa."
 		(exclude_from_sim no)
-		(at 151.13 57.15 0)
+		(at 151.13 55.88 0)
 		(effects
 			(font

Commit message: chore(hw): tidy and set ${REVISION} to "B"
Other:
- company: https://is.gd/6hpvh6 -> https://tinyurl.com/econopet-rev-b
Changed lines of the file:
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@@
 	(title_block
 		(title "EconoPET 40/8096")
-		(date "2026-02-27")
-		(rev "B")
-		(company "https://is.gd/6hpvh6")
+		(date "2026-08-25")
+		(rev "${REVISION}")
+		(company "https://tinyurl.com/econopet-rev-b")
 		(comment 1 "Unspecified resistors are 1% / 62.5mW")
 		(comment 2 "Unspecified capacitors are 25V")

Commit message: chore(hw): create production files
Parts:
- C67, C68, C69: LCSC C307331 -> (none); LCSC Part # (none) -> C307331
- R38: LCSC C11702 -> (none); LCSC Part # (none) -> C11702
Changed lines of the file:
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@@
+			)
+		)
+		(property "FT Position Offset" ""
+			(at 86.36 153.67 0)
+			(effects
+				(font
+					(size 1.27 1.27)
+				)
+				(hide yes)
+			)
+		)
+		(property "FT Rotation Offset" ""
+			(at 86.36 153.67 0)
+			(effects
+				(font
+					(size 1.27 1.27)
+				)
+				(hide yes)
 			)
 		)
@@
 			)
 		)
+		(property "FT Position Offset" ""
+			(at 184.15 128.27 0)
+			(effects
+				(font
+					(size 1.27 1.27)
+				)
+				(hide yes)
+			)
+		)
+		(property "FT Rotation Offset" ""
+			(at 184.15 128.27 0)
+			(effects
+				(font
+					(size 1.27 1.27)
+				)
+				(hide yes)
+			)
+		)
 		(pin "1"
 		)
@@
 			)
 		)
+		(property "FT Position Offset" ""
+			(at 86.36 58.42 0)
+			(effects
+				(font
+					(size 1.27 1.27)
+				)
+				(hide yes)
+			)
+		)
+		(property "FT Rotation Offset" ""
+			(at 86.36 58.42 0)
+			(effects
+				(font
+					(size 1.27 1.27)
+				)
+				(hide yes)
+			)
+		)
 		(pin "1"
 		)
@@
 			)
 		)
-		(property "LCSC" "C307331"
+		(property "LCSC Part #" "C307331"
+			(at 97.79 118.11 0)
+			(effects
+				(font
+					(size 1.27 1.27)
+				)
+				(hide yes)
+			)
+		)
+		(property "FT Position Offset" ""
+			(at 97.79 118.11 0)
+			(effects
+				(font
+					(size 1.27 1.27)
+				)
+				(hide yes)
+			)
+		)
+		(property "FT Rotation Offset" ""
 			(at 97.79 118.11 0)
 			(effects
@@
 			)
 		)
-		(property "LCSC" "C307331"
+		(property "LCSC Part #" "C307331"
+			(at 100.33 22.86 0)
+			(effects
+				(font
+					(size 1.27 1.27)
+				)
+				(hide yes)
+			)
+		)
+		(property "FT Position Offset" ""
+			(at 100.33 22.86 0)
+			(effects
+				(font
+					(size 1.27 1.27)
+				)
+				(hide yes)
+			)
+		)
+		(property "FT Rotation Offset" ""
 			(at 100.33 22.86 0)
 			(effects
@@
 			)
 		)
-		(property "LCSC" "C307331"
+		(property "LCSC Part #" "C307331"
+			(at 198.12 91.44 0)
+			(effects
+				(font
+					(size 1.27 1.27)
+				)
+				(hide yes)
+			)
+		)
+		(property "FT Position Offset" ""
+			(at 198.12 91.44 0)
+			(effects
+				(font
+					(size 1.27 1.27)
+				)
+				(hide yes)
+			)
+		)
+		(property "FT Rotation Offset" ""
 			(at 198.12 91.44 0)
 			(effects
@@
 			)
 		)
-		(property "LCSC" "C11702"
+		(property "LCSC Part #" "C11702"
 			(at 227.33 143.51 0)
 			(effects
+				(font
+					(size 1.27 1.27)
+				)
+				(hide yes)
+			)
+		)
+		(property "FT Position Offset" ""
+			(at 227.33 143.51 0)
+			(effects
+				(font
+					(size 1.27 1.27)
+				)
+				(hide yes)
+			)
+		)
+		(property "FT Rotation Offset" ""
+			(at 227.33 143.51 0)
+			(effects

Commit message: feat(hw): separate PHI2 clock for PIA1
Connections:
- net BPHI2: no longer U11.25 (ϕ2)
- new net BPHI2_PIA1: U11.25 (ϕ2)
Changed lines of the file:
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@@
-	(wire
-		(pts
-			(xy 71.12 33.02) (xy 41.91 33.02)
-		)
-		(stroke
-			(width 0)
-			(type default)
-		)
-	)
 	(wire
 		(pts
@@
 	(wire
 		(pts
-			(xy 41.91 33.02) (xy 41.91 102.87)
-		)
-		(stroke
-			(width 0)
-			(type default)
-		)
-	)
-	(wire
-		(pts
 			(xy 69.85 38.1) (xy 44.45 38.1)
 		)
@@
 		(pts
 			(xy 111.76 33.02) (xy 101.6 33.02)
+		)
+		(stroke
+			(width 0)
+			(type default)
+		)
+	)
+	(wire
+		(pts
+			(xy 30.48 33.02) (xy 71.12 33.02)
 		)
 		(stroke
@@
 		)
 	)
+	(hierarchical_label "BPHI2_PIA1"
+		(shape input)
+		(at 30.48 33.02 180)
+		(fields_autoplaced yes)
+		(effects
+			(font
+				(size 1.27 1.27)
+			)
+			(justify right)
+		)
+	)
