File: hw/rev-b/mainboard/kicad/Mainboard.kicad_sch (KiCad schematic)
At the start: 0 parts

Commit message: hw: label JIFFY signal, tidy stitching
Other:
- sheet IO ports: added BJIFFY; removed BVSYNC
- sheet MAGIC ports: added BJIFFY; removed BVSYNC
Changed lines of the file:
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@@
-			)
-		)
-		(pin "BVSYNC" output
-			(at 104.14 127 0)
-			(effects
-				(font
-					(size 1.27 1.27)
-				)
-				(justify right)
 			)
 		)
@@
 				)
 				(justify left)
+			)
+		)
+		(pin "BJIFFY" output
+			(at 104.14 127 0)
+			(effects
+				(font
+					(size 1.27 1.27)
+				)
+				(justify right)
 			)
 		)
@@
 			)
 		)
-		(pin "BVSYNC" input
+		(pin "BJIFFY" input
 			(at 116.84 127 180)
 			(effects

Commit message: chore(hw): tidy and set ${REVISION} to "B"
Other:
- company: https://is.gd/6hpvh6 -> https://tinyurl.com/econopet-rev-b
Changed lines of the file:
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@@
 	(title_block
 		(title "EconoPET 40/8096")
-		(date "2026-02-27")
-		(rev "B")
-		(company "https://is.gd/6hpvh6")
+		(date "2026-08-25")
+		(rev "${REVISION}")
+		(company "https://tinyurl.com/econopet-rev-b")
 		(comment 1 "Unspecified resistors are 1% / 62.5mW")
 		(comment 2 "Unspecified capacitors are 25V")

Commit message: feat(hw): separate audio_l / audio_r (schematic only)
Other:
- sheet AUDIO ports: added AUDIO_L, AUDIO_R; removed AUDIO
- sheet MAGIC ports: added AUDIO_L, AUDIO_R; removed AUDIO
Changed lines of the file:
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@@
+	(wire
+		(pts
+			(xy 66.04 121.92) (xy 78.74 121.92)
+		)
+		(stroke
+			(width 0)
+			(type default)
+		)
+	)
 	(wire
 		(pts
@@
 			)
 		)
-		(pin "AUDIO" output
-			(at 78.74 119.38 180)
-			(effects
-				(font
-					(size 1.27 1.27)
-				)
-				(justify left)
-			)
-		)
 		(pin "~{AUDIO_DET}" input
 			(at 78.74 116.84 180)
@@
 				)
 				(justify right)
+			)
+		)
+		(pin "AUDIO_R" output
+			(at 78.74 121.92 180)
+			(effects
+				(font
+					(size 1.27 1.27)
+				)
+				(justify left)
+			)
+		)
+		(pin "AUDIO_L" output
+			(at 78.74 119.38 180)
+			(effects
+				(font
+					(size 1.27 1.27)
+				)
+				(justify left)
 			)
 		)
@@
 	(sheet
 		(at 40.64 113.03)
-		(size 25.4 10.16)
+		(size 25.4 12.7)
 		(fields_autoplaced yes)
 		(stroke
@@
 		)
 		(property "Sheetfile" "Audio.kicad_sch"
-			(at 40.64 123.7746 0)
+			(at 40.64 126.3146 0)
 			(effects
 				(font
@@
 				)
 				(justify left top)
-			)
-		)
-		(pin "AUDIO" input
-			(at 66.04 119.38 0)
-			(effects
-				(font
-					(size 1.27 1.27)
-				)
-				(justify right)
 			)
 		)
@@
 			(effects
 				(font
+					(size 1.27 1.27)
+				)
+				(justify right)
+			)
+		)
+		(pin "AUDIO_R" input
+			(at 66.04 121.92 0)
+			(effects
+				(font
+					(size 1.27 1.27)
+				)
+				(justify right)
+			)
+		)
+		(pin "AUDIO_L" input
+			(at 66.04 119.38 0)
+			(effects
+				(font

Commit message: feat(hw): separate PHI2 clock for PIA1
Other:
- sheet IO ports: added BPHI2_PIA1; removed none
- sheet MAGIC ports: added BPHI2_PIA1; removed none
Changed lines of the file:
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@@
+	(wire
+		(pts
+			(xy 104.14 110.49) (xy 116.84 110.49)
+		)
+		(stroke
+			(width 0)
+			(type default)
+		)
+	)
 	(wire
 		(pts
@@
 			)
 		)
+		(pin "BPHI2_PIA1" output
+			(at 104.14 110.49 0)
+			(effects
+				(font
+					(size 1.27 1.27)
+				)
+				(justify right)
+			)
+		)
 		(instances
 			(project "Mainboard"
@@
 			(effects
 				(font
+					(size 1.27 1.27)
+				)
+				(justify left)
+			)
+		)
+		(pin "BPHI2_PIA1" input
+			(at 116.84 110.49 180)
+			(effects
+				(font
