File: hw/rev-b/mainboard/kicad/DVI.kicad_sch (KiCad schematic)
At the start: 14 parts, among them J24 NOT_HDMI_A

Commit message: chore(hw): tidy and set ${REVISION} to "B"
Other:
- company: https://is.gd/6hpvh6 -> https://tinyurl.com/econopet-rev-b
Changed lines of the file:
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@@
 	(title_block
 		(title "EconoPET 40/8096")
-		(date "2026-02-27")
-		(rev "B")
-		(company "https://is.gd/6hpvh6")
+		(date "2026-08-25")
+		(rev "${REVISION}")
+		(company "https://tinyurl.com/econopet-rev-b")
 		(comment 1 "Unspecified resistors are 1% / 62.5mW")
 		(comment 2 "Unspecified capacitors are 25V")

Commit message: chore(hw): create production files
Parts:
- C99: LCSC C23733 -> (none); LCSC Part # (none) -> C23733
- J24: FT Rotation Offset (none) -> 90; LCSC C138388 -> (none); LCSC Part # (none) -> C138388
- R50, R51, R52: LCSC C25879 -> (none); LCSC Part # (none) -> C25879
- R53, R54, R55, R56, R57, R58, R59, R60, R61: LCSC C22966 -> (none); LCSC Part # (none) -> C22966

Commit message: fix(hw): remove I2C0 jumpers
Connections:
- net SCL: no longer names the net of J24.15 (SCL), R51.2
- net SDA: no longer names the net of J24.16 (SDA), R52.2
Other:
- note removed: "CEC, SCL, and SDA are for experimentation and disconnected by solder jumpers by default. DANGER: Closing the DVI_SCL/DVI_SDA jumpers pulls the corresponding RP2040 GPIO pins to +5V. Only do this if you know what you're doing."
Changed lines of the file:
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@@
-	)
-	(junction
-		(at 121.92 113.03)
-		(diameter 0)
-		(color 0 0 0 0)
 	)
 	(junction
@@
 	)
 	(junction
-		(at 116.84 102.87)
-		(diameter 0)
-		(color 0 0 0 0)
-	)
-	(junction
 		(at 185.42 119.38)
 		(diameter 0)
@@
 	(wire
 		(pts
-			(xy 154.94 113.03) (xy 154.94 100.33)
-		)
-		(stroke
-			(width 0)
-			(type default)
-		)
-	)
-	(wire
-		(pts
 			(xy 121.92 60.96) (xy 177.8 60.96)
 		)
@@
 	(wire
 		(pts
-			(xy 85.09 102.87) (xy 116.84 102.87)
-		)
-		(stroke
-			(width 0)
-			(type default)
-		)
-	)
-	(wire
-		(pts
 			(xy 200.66 60.96) (xy 200.66 59.69)
 		)
@@
 	(wire
 		(pts
-			(xy 151.13 102.87) (xy 151.13 97.79)
-		)
-		(stroke
-			(width 0)
-			(type default)
-		)
-	)
-	(wire
-		(pts
 			(xy 182.88 119.38) (xy 185.42 119.38)
 		)
@@
 	(wire
 		(pts
-			(xy 85.09 113.03) (xy 121.92 113.03)
-		)
-		(stroke
-			(width 0)
-			(type default)
-		)
-	)
-	(wire
-		(pts
 			(xy 149.86 85.09) (xy 135.89 85.09)
 		)
@@
 	(wire
 		(pts
-			(xy 116.84 87.63) (xy 116.84 102.87)
+			(xy 116.84 87.63) (xy 116.84 97.79)
 		)
 		(stroke
@@
 	(wire
 		(pts
-			(xy 151.13 97.79) (xy 167.64 97.79)
-		)
-		(stroke
-			(width 0)
-			(type default)
-		)
-	)
-	(wire
-		(pts
-			(xy 121.92 87.63) (xy 121.92 113.03)
+			(xy 121.92 87.63) (xy 121.92 100.33)
 		)
 		(stroke
@@
 	(wire
 		(pts
-			(xy 154.94 100.33) (xy 167.64 100.33)
-		)
-		(stroke
-			(width 0)
-			(type default)
-		)
-	)
-	(wire
-		(pts
 			(xy 154.94 92.71) (xy 167.64 92.71)
 		)
@@
 	(wire
 		(pts
-			(xy 121.92 113.03) (xy 154.94 113.03)
+			(xy 121.92 100.33) (xy 167.64 100.33)
 		)
 		(stroke
@@
 	(wire
 		(pts
-			(xy 116.84 102.87) (xy 151.13 102.87)
+			(xy 116.84 97.79) (xy 167.64 97.79)
 		)
 		(stroke
@@
 		)
 	)
-	(text "CEC, SCL, and SDA are for experimentation and\ndisconnected by solder jumpers by default.\n\nDANGER: Closing the DVI_SCL/DVI_SDA jumpers pulls\nthe corresponding RP2040 GPIO pins to +5V.\n\nOnly do this if you know what you're doing."
-		(exclude_from_sim no)
-		(at 80.01 134.62 0)
-		(effects
-			(font
-				(size 1.27 1.27)
-			)
-			(justify left bottom)
-		)
-	)
 	(text "DVI TMDS protocol over an HDMI-compatible\nconnector (not HDMI certified).\n\nSee: https://github.com/Wren6991/PicoDVI"
 		(exclude_from_sim no)
@@
 		)
 	)
-	(hierarchical_label "SCL"
-		(shape input)
-		(at 85.09 102.87 180)
-		(fields_autoplaced yes)
-		(effects
-			(font
-				(size 1.27 1.27)
-			)
-			(justify right)
-		)
-	)
 	(hierarchical_label "{DVI}"
 		(shape input)
@@
 		(fields_autoplaced yes)
 		(effects
-			(font
-				(size 1.27 1.27)
-			)
-			(justify right)
-		)
-	)
-	(hierarchical_label "SDA"
-		(shape bidirectional)
-		(at 85.09 113.03 180)
-		(fields_autoplaced yes)
-		(effects
